File: Schematics/Communications_Module/Communications_Module.kicad_pcb (KiCad board)
At the start: 4 copper layers, 69.5 x 60 mm, 74 parts, among them J1 USB_C_Female_USB2_Small, J2 SWD_01x04_Pin, J3 Stack Male Edge Connector, Q1 AO3400A, SW1 SW_STM_RESET, SW2 SW_STM_BOOT_MODE, U1 RFM95W-915, U2 W25Q128JVS, U3 AMS1117-3.3, U4 LM66100DCKR, U5 LM66100DCKR, U6 LM66100DCKR, U7 STM32F103CBT6, U8 ACS70331EOLC, U9 ISO1042BDWVR, Y1 X322516MMB4SI

Commit message: Very minor PCB tweaks
Routing:
- net V_MUX: track 127.0 -> 125.1 mm
- net +5V: track 31.8 -> 32.4 mm
Other:
- board text removed: "-->"
- board text removed: "IDK what to do about these ground pins"
Changed lines of the file:
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@@
-    (effects (font (size 1 1) (thickness 0.15)) (justify left bottom))
-  )
-  (gr_text "-->" (at 143.9 70.6 -90) (layer "Cmts.User")
     (effects (font (size 1 1) (thickness 0.15)) (justify left bottom))
   )
   (gr_text "USE GRID THAT IS SOME\nMULTIPLE OF 0.1mm\n\n(0.1mm, 0.2mm, 0.5mm, 1.0mm, etc)" (at 177.6 133.2) (layer "Cmts.User")
-    (effects (font (size 1 1) (thickness 0.15)) (justify left bottom))
-  )
-  (gr_text "IDK what to do about these ground pins" (at 132.3 70.5) (layer "Cmts.User")
     (effects (font (size 1 1) (thickness 0.15)) (justify left bottom))
   )
@@
   (segment (start 133.495 92.76) (end 133.495 90.51) (width 0.5) (layer "F.Cu") (net 3))
   (via (at 130.725 86.027707) (size 0.7) (drill 0.3) (layers "F.Cu" "B.Cu") (net 3))
-  (segment (start 145.5 79.85) (end 144.5 80.85) (width 0.5) (layer "B.Cu") (net 3))
-  (segment (start 145.5 78.2) (end 145.5 79.85) (width 0.5) (layer "B.Cu") (net 3))
   (segment (start 139.35 86) (end 130.752707 86) (width 0.5) (layer "B.Cu") (net 3))
+  (segment (start 145.5 78.2) (end 145.5 80.85) (width 0.5) (layer "B.Cu") (net 3))
   (segment (start 144.5 80.85) (end 139.35 86) (width 0.5) (layer "B.Cu") (net 3))
+  (segment (start 145.5 80.85) (end 144.5 80.85) (width 0.5) (layer "B.Cu") (net 3))
   (segment (start 144.5 78.2) (end 144.5 80.85) (width 0.5) (layer "B.Cu") (net 3))
   (segment (start 130.752707 86) (end 130.725 86.027707) (width 0.5) (layer "B.Cu") (net 3))
@@
   (segment (start 171.05 95.75) (end 171.1 95.8) (width 1) (layer "F.Cu") (net 27))
   (segment (start 169.5 118.2) (end 171.1 116.6) (width 0.5) (layer "F.Cu") (net 27))
-  (segment (start 171.1 88.65) (end 171.1 86.8) (width 1) (layer "F.Cu") (net 27))
   (segment (start 163.05 106.5) (end 163.7 105.85) (width 0.5) (layer "F.Cu") (net 27))
   (segment (start 168.4 84.1) (end 162.45 84.1) (width 1) (layer "F.Cu") (net 27))

Commit message: Final Revisions
Routing:
- net +3.3V: track 437.5 -> 397.0 mm
Changed lines of the file:
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@@
     (property "ki_keywords" "test point tp")
     (attr exclude_from_pos_files exclude_from_bom)
-    (fp_text reference "TP9" (at 0 -1.75) (layer "F.SilkS")
+    (fp_text reference "TP9" (at 0.2 -1.75) (layer "F.SilkS")
         (effects (font (size 0.8 0.8) (thickness 0.1)))
     )
@@
     (property "ki_keywords" "test point tp")
     (attr exclude_from_pos_files exclude_from_bom)
-    (fp_text reference "TP11" (at -0.05 -1.75) (layer "F.SilkS")
+    (fp_text reference "TP11" (at 0.15 -1.75) (layer "F.SilkS")
         (effects (font (size 0.8 0.8) (thickness 0.1)))
     )
@@
   (segment (start 167.1 95.44) (end 167.1 90.6) (width 1) (layer "B.Cu") (net 24))
   (segment (start 160.6 111.45) (end 160.35 111.2) (width 0.3) (layer "B.Cu") (net 24))
+  (segment (start 131.55 88.85) (end 128.4 85.7) (width 0.5) (layer "B.Cu") (net 24))
   (segment (start 148.54 120.51) (end 153.65 120.51) (width 0.5) (layer "B.Cu") (net 24))
   (segment (start 167.1 120.52) (end 167.1 119.88) (width 1) (layer "B.Cu") (net 24))
@@
   (segment (start 167.1 105.5) (end 167.1 102) (width 1) (layer "B.Cu") (net 24))
   (segment (start 149.968629 97.1) (end 150.668629 97.8) (width 0.5) (layer "B.Cu") (net 24))
+  (segment (start 127.402082 85.7) (end 126.342082 84.64) (width 0.5) (layer "B.Cu") (net 24))
   (segment (start 142.05 125.55) (end 143.5 125.55) (width 0.5) (layer "B.Cu") (net 24))
   (segment (start 152.7 104.7) (end 167 104.7) (width 1) (layer "B.Cu") (net 24))
+  (segment (start 128.4 85.7) (end 127.402082 85.7) (width 0.5) (layer "B.Cu") (net 24))
   (segment (start 167 110.4) (end 167.1 110.3) (width 0.5) (layer "B.Cu") (net 24))
   (segment (start 160.35 111.2) (end 162.8 111.2) (width 0.5) (layer "B.Cu") (net 24))
@@
   (segment (start 167 90.5) (end 167.1 90.6) (width 0.5) (layer "B.Cu") (net 24))
   (segment (start 153.8 120.36) (end 153.65 120.51) (width 0.5) (layer "B.Cu") (net 24))
-  (segment (start 128.4 85.7) (end 131.55 88.85) (width 0.5) (layer "B.Cu") (net 24))
   (segment (start 167.1 119.88) (end 167.1 116.7) (width 1) (layer "B.Cu") (net 24))
   (segment (start 133.834925 117.85) (end 137.334925 114.35) (width 1) (layer "B.Cu") (net 24))
@@
   (segment (start 152 112.5) (end 154.1 110.4) (width 0.5) (layer "B.Cu") (net 24))
   (segment (start 147 112.5) (end 152 112.5) (width 0.5) (layer "B.Cu") (net 24))
-  (segment (start 126.342082 84.64) (end 131.282082 89.58) (width 0.5) (layer "B.Cu") (net 24))
   (segment (start 148.47 93.86) (end 166.83 93.86) (width 0.5) (layer "B.Cu") (net 24))
-  (segment (start 166.75 89.58) (end 167.1 89.93) (width 0.5) (layer "B.Cu") (net 24))
-  (segment (start 131.282082 89.58) (end 166.75 89.58) (width 0.5) (layer "B.Cu") (net 24))
   (segment (start 154.9 123.5) (end 158.05 123.5) (width 0.5) (layer "F.Cu") (net 25))
   (segment (start 163 118.2) (end 161.5 118.2) (width 0.5) (layer "F.Cu") (net 25))
