File: Schematics/Sensors_Module/Sensors_Module.kicad_sch (KiCad schematic)
At the start: 0 parts

Commit message: Needs Review but mostly done apart from a few pins on the MCU
Parts:
- added BZ1: PKM13EPYH4000-A0, symbol Device:Buzzer
- added C1 (x2): 100n, symbol Device:C
- added C1, C16, C2: 0.1u, symbol Device:C
- added C13: 104, symbol Device:C
- added C14, C16, C17, C18: 0.1uF, symbol Device:C
- added C15: 1000u, symbol Device:C
- added C15: 1uF, symbol Device:C
- added C19: C-Filter, symbol Device:C
- added C2, C3: 10μF, symbol Device:C
- added C4, C7: 9p, symbol Device:C
- added C5, C6, C8: 1u, symbol Device:C
- added C7: 2.2uF, symbol Device:C
- added D1: PWR_LED, symbol Device:LED
- added D2, D3: D, symbol Device:D
- added D4: WS2812B, LED_SMD:LED_WS2812B_PLCC4_5.0x5.0mm_P3.2mm, symbol LED:WS2812B
- added J1: USB_B_Micro, symbol Connector:USB_B_Micro
- added J2: Stack Male Edge Connector, Connector_PCBEdge:BUS_PCIexpress_x1, symbol QRET_Edge_Connector:Stack Male Edge Connector
- added J3: Conn_01x04_Pin, symbol Connector:Conn_01x04_Pin
- added NAU7802: ~, symbol Libary:NAU7802
- added Q1: NMOS, symbol Simulation_SPICE:NMOS
- added R1 (x2): 2.7k, symbol Device:R_US
- added R1, R3, R5, R7: 10k, symbol Device:R_US
- added R4: 500, symbol Device:R_US
- added R6 (x7), R9: 1k, symbol Device:R_US
- added R8: 1.5k, symbol Device:R_US
- added SW1: Boot Mode, symbol Switch:SW_SPDT
- added U1: STM32F103CBTx, Package_QFP:LQFP-48_7x7mm_P0.5mm, symbol MCU_ST_STM32F1:STM32F103CBTx
- added U2: W25Q128JVSIQ, symbol Memory_Flash:W25Q128JVS
- added U3: AMS1117-3.3, Package_TO_SOT_SMD:SOT-223-3_TabPin2, symbol Regulator_Linear:AMS1117-3.3
- added U4, U5, U6: LM66100DCKR, DCK6_TEX, symbol QRET_Buck_PSU:LM66100DCKR
- added U8: MMC5633NJL, Package_BGA:WLP-4_0.86x0.86mm_P0.4mm, symbol Sensor_Magnetic:MMC5633NJL
- added U8: ACS706xLC-05C, symbol Sensor_Current:ACS706xLC-05C
- added U9: ISO1042BQDWVQ1, symbol QRET_CANBUS:ISO1042BQDWVQ1
- added Y1: X322516MMB4SI, symbol Device:Crystal_GND24
Connections:
- new net: BZ1.1 (-), D2.1 (K), D3.1 (K), R6.1
- new net: C7.2, U8.A1 (VSA)
- new net: R1.2, U8.A2 (SCL)
- new net: R1.1, U8.B2 (SDA)
- new net: C1.2, U9.8 (VCC2)
- new net: D1.2 (A), R9.2
- new net: C14.1, NAU7802.6 (VBG)
- new net: BZ1.2 (+), Q1.1 (D), R6.2
- new net: C16.1, C17.1, NAU7802.1 (REFP), NAU7802.16 (AVDD), R6.1, R6.2
- new net: C1.1, U1.7 (NRST)
- new net: J2.A1 (BATT_A), J2.A2 (BATT_A), J2.B1 (BATT_A), J2.B2 (BATT_A)
- new net: J2.A10 (BATT_B), J2.A9 (BATT_B), J2.B10 (BATT_B), J2.B9 (BATT_B)
- new net: J2.A11 (GND_B), J2.A12 (GND_B), J2.A14 (GND_B), J2.B11 (GND_B), J2.B12 (GND_B), J2.B14 (GND_B)
- new net: J2.A13 (3.3V_B), J2.B13 (3.3V_B)
- new net: J2.A5 (3.3V_A), J2.B5 (3.3V_A)
- new net: Q1.2 (G), R4.2, R5.1
- new net: R7.1, SW1.2 (B)
- new net: R3.2, U2.3 (IO2)
- new net: C18.1, NAU7802.2 (VIN1N), R6.2
- new net: C18.2, NAU7802.3 (VIN1P), R6.2
- new net: C19.1, NAU7802.4 (VIN2N)
- new net: C19.2, NAU7802.5 (VIN2P)
- new net: R6.1, R6.1, R6.2
- new net: R6.1, R6.1, R6.1
- new net +3.3V: C1.1, C13.1, C15.1, C2.2, C7.1, D2.2 (A), D4.1 (VDD), NAU7802.15 (DVDD), R1.1, R3.1, R8.1, R9.1, SW1.3 (C), U1.1 (VBAT), U1.24 (VDD), U1.36 (VDD), U1.48 (VDD), U2.8 (VCC), U8.3 (IP-), U8.4 (IP-), U8.B1 (VDD), U9.1 (VCC1)
- new net +3.3VA: U1.9 (VDDA)
- new net +5V: J2.A7 (5.0V_A), J2.B7 (5.0V_A)
- new net BOOT0: R7.2, U1.44 (BOOT0)
- new net CAN_H: J2.A15 (CAN_H)
- new net CAN_L: J2.B15 (CAN_L)
- new net CAN_RX: U1.45 (PB8), U9.3 (RXD)
- new net CAN_TX: U1.46 (PB9), U9.2 (TXD)
- new net CS_FL: U1.25 (PB12), U2.1 (~{CS})
- new net D+: J1.3 (D+), R8.2, U1.33 (PA12)
- new net D-: J1.2 (D-), U1.32 (PA11)
- new net GND: C1.2, C1.2, C13.2, C14.2, C15.2, C15.2, C16.2, C16.2, C17.2, C2.1, C2.2, C3.2, C4.2, C5.2, C6.2, C7.2, C8.2, D1.1 (K), D4.3 (VSS), J1.5 (GND), J2.A3 (GND_A), J2.A4 (GND_A), J2.A6 (GND_A), J2.A8 (GND_A), J2.B3 (GND_A), J2.B4 (GND_A), J2.B6 (GND_A), J2.B8 (GND_A), J3.1 (Pin_1), NAU7802.7 (REFN), NAU7802.8 (AVSS), NAU7802.9 (DVSS), Q1.3 (S), R5.2, R6.2, R6.2, SW1.1 (A), U1.23 (VSS), U1.35 (VSS), U1.47 (VSS), U1.8 (VSSA), U2.4 (GND), U3.1 (GND), U4.2 (GND), U4.5 (ST), U5.2 (GND), U5.5 (ST), U6.2 (GND), U6.5 (ST), U8.5 (GND), U9.4 (GND1), Y1.2, Y1.4
- new net GND2: C1.1, U9.5 (GND2)
- new net MISO_FL: U1.27 (PB14), U2.2 (DO(IO1))
- new net MOSI_FL: U1.28 (PB15), U2.5 (DI(IO0))
- new net OSC_IN: C4.1, U1.5 (PD0), Y1.1
- new net OSC_OUT: C7.1, U1.6 (PD1), Y1.3
- new net RESET_FL: R1.2, U1.29 (PA8), U2.7 (IO3)
- new net RGB: D4.4 (DIN)
- new net SCK_FL: U1.26 (PB13), U2.6 (CLK)
- new net SDCLK: U1.37 (PA14)
- new net SWCLK: J3.2 (Pin_2)
- new net SWDIO: J3.3 (Pin_3), U1.34 (PA13)
- new net V_BATT: D3.2 (A)
- new net V_BUZZ: R4.1, U1.30 (PA9)
- new net V_CLK: NAU7802.13 (SCLK), U1.13 (PA3)
- new net V_DI: NAU7802.14 (SDIO), U1.11 (PA1)
- new net V_DIODE: C15.1, C16.1, U4.3 (*CE), U4.6 (VOUT), U5.3 (*CE), U5.6 (VOUT), U6.3 (*CE), U6.6 (VOUT), U8.1 (IP+), U8.2 (IP+), U8.8 (VCC)
- new net V_DR: NAU7802.12 (DRDY), U1.12 (PA2)
- new net V_Isense: U1.10 (PA0), U8.7 (VOUT)
- new net V_MAG: R1.1, R1.2, U1.41 (PB5)
- new net V_PSU: C5.1, U4.1 (VIN)
- new net V_REG: C3.1, C8.1, U3.2 (VO), U5.1 (VIN)
- new net V_SWD: C6.1, J3.4 (Pin_4), U6.1 (VIN)
- new net V_USB: C2.1, J1.1 (VBUS), U3.3 (VI)
- no-connect marks 0 -> 10
Other:
- note added: "-> go to connectors ->"
- note added: "Also SPI no ic2"
- note added: "Be wary of the resistor count (depending on how many sensors)"
- note added: "Boot Mode"
- note added: "Buzzer"
- note added: "CANBUS"
- note added: "Capacitor to prevent unintended resets"
- note added: "Crystal Oscillator"
- note added: "Current Sense + 3.3V output"
- note added: "Flash Module"
- note added: "Galvanic isolation barrier"
- note added: "HIGH = PROGRAMMING MODE LOW = RUN MEMORY"
- note added: "Ideal Diodes"
- note added: "Load Cell and ADC"
- note added: "Magnetometer"
- note added: "Maybe?"
- note added: "Need iso GND, and iso power supply VCC2 range: 4.5 > VCC2 > 5.5"
- note added: "RGB Indicator"
- note added: "ST pins are just status indication, Want a way to keep track of what power supply active?"
- note added: "Serial Wire Debug"
- note added: "Stack Edge Connector"
- note added: "Stack Edge Connector needs a capacitor where the 3.3 volt is comming directly off"
- note added: "To Do: -Flash Module -Magnotometer -Music -Light Sensor (LDR, photoresistor) -Boot and Reset Buttons"
- note added: "USB"
- note added: "Units? (Capacitors) -ID"
- note added: "can u use the same pullup?"
- note added: "needed if same node as 1000u?"

Commit message: Update Sensors_Module.kicad_sch
Parts:
- removed C1 (x2): 100n, symbol Device:C
- removed C1, C16, C2: 0.1u, symbol Device:C
- removed C14, C16: 0.1uF, symbol Device:C
- removed C15: 1000u, symbol Device:C
- removed C15: 1uF, symbol Device:C
- removed C19: C-Filter, symbol Device:C
- removed C2: 10μF, symbol Device:C
- removed C7: 2.2uF, symbol Device:C
- removed C7: 9p, symbol Device:C
- removed D3: D, symbol Device:D
- removed NAU7802: ~, symbol Libary:NAU7802
- removed R1 (x2): 2.7k, symbol Device:R_US
- removed R1: 10k, symbol Device:R_US
- removed R6 (x7): 1k, symbol Device:R_US
- removed U8: MMC5633NJL, Package_BGA:WLP-4_0.86x0.86mm_P0.4mm, symbol Sensor_Magnetic:MMC5633NJL
- added C1 (x2): 100n, symbol Device:C
- added C1, C16, C2: 0.1u, symbol Device:C
- added C11: 2.2uF, symbol Device:C
- added C15: 1000u, symbol Device:C
- added C16: 0.1uF, symbol Device:C
- added C2: 10μF, symbol Device:C
- added C20, C21: 1uF, symbol Device:C
- added C7: 9p, symbol Device:C
- added D1: D, symbol Device:D
- added J4: Screw_Terminal_01x02, symbol Connector:Screw_Terminal_01x02
- added J5: Screw_Terminal, symbol Connector:Screw_Terminal_01x02
- added JP1: Jumper_2_Bridged, symbol Jumper:Jumper_2_Bridged
- added NAU1: ~, symbol Libary:NAU7802
- added R1 (x2): 2.7k, symbol Device:R_US
- added R1: 10k, symbol Device:R_US
- added R6 (x3): 1k, symbol Device:R_US
- added R6 (x4): 47k, symbol Device:R_US
- added U4: MMC5633NJL, Package_BGA:WLP-4_0.86x0.86mm_P0.4mm, symbol Sensor_Magnetic:MMC5633NJL
Connections:
- net +3.3V: now also C1.1, C11.1, C2.2, C21.1, NAU1.15 (DVDD), R1.1, U4.B1 (VDD)
- net GND: now also C18.2, C1.2, C1.2, C15.2, C16.1, C16.2, C16.2, C2.1, C2.2, C20.1, C20.2, C21.2, C7.2, J4.1 (Pin_1), J4.2 (Pin_2), JP1.2 (B), NAU1.1 (REFP), NAU1.16 (AVDD), NAU1.7 (REFN), NAU1.8 (AVSS), NAU1.9 (DVSS), R6.1, R6.1, R6.2; no longer C17.2
- net GND2: now also C1.1
- net OSC_OUT: now also C7.1
- net RESET_FL: now also R1.2
- net V_BATT: now also D1.2 (A)
- net V_CLK: now also NAU1.13 (SCLK)
- net V_DI: now also NAU1.14 (SDIO)
- net V_DIODE: now also C15.1, C16.1
- net V_DR: now also NAU1.12 (DRDY)
- net V_MAG: now also R1.1, R1.2
- net V_USB: now also C2.1
- net at BZ1.1 (-), D2.1 (K): now also D1.1 (K), R6.1
- net at U9.8 (VCC2): now also C1.2
- net at BZ1.2 (+), Q1.1 (D): now also R6.2
- net at C17.1: now also NAU1.2 (VIN1N), R6.2
- net at U1.7 (NRST): now also C1.1
- net at C18.1: now also NAU1.6 (VBG)
- new net: C11.2, U4.A1 (VSA)
- new net: R1.2, U4.A2 (SCL)
- new net: R1.1, U4.B2 (SDA)
- new net: C17.2, NAU1.3 (VIN1P), R6.2
- new net: R6.1, R6.1, R6.2
- new net: J5.2 (Pin_2), JP1.1 (A), NAU1.4 (VIN2N), R6.2
- new net: J5.1 (Pin_1), R6.2
- new net: NAU1.5 (VIN2P), R6.1, R6.1
Other:
- note added: "Put on one of the sides (really small and hard to soder)"

Commit message: Various changes
-Added many symbols and footprints
-Pulled base changes from other schematics
-Organized schematic
-Added attribution text
Parts:
- removed BZ1: PKM13EPYH4000-A0, symbol Device:Buzzer
- removed C1: 100n, symbol Device:C
- removed C1, C16, C2: 0.1u, symbol Device:C
- removed C13: 104, symbol Device:C
- removed C15: 1000u, symbol Device:C
- removed C2, C3: 10μF, symbol Device:C
- removed C5: 1u, symbol Device:C
- removed D1, D2: D, symbol Device:D
- removed J1: USB_B_Micro, symbol Connector:USB_B_Micro
- removed J2: Stack Male Edge Connector, Connector_PCBEdge:BUS_PCIexpress_x1, symbol QRET_Edge_Connector:Stack Male Edge Connector
- removed J3: Conn_01x04_Pin, symbol Connector:Conn_01x04_Pin
- removed Q1: NMOS, symbol Simulation_SPICE:NMOS
- removed R1, R3, R5, R7: 10k, symbol Device:R_US
- removed R4: 500, symbol Device:R_US
- removed R6, R9: 1k, symbol Device:R_US
- removed R8: 1.5k, symbol Device:R_US
- removed SW1: Boot Mode, symbol Switch:SW_SPDT
- removed U2: W25Q128JVSIQ, symbol Memory_Flash:W25Q128JVS
- removed U3: AMS1117-3.3, Package_TO_SOT_SMD:SOT-223-3_TabPin2, symbol Regulator_Linear:AMS1117-3.3
- removed U4, U5, U6: LM66100DCKR, DCK6_TEX, symbol QRET_Buck_PSU:LM66100DCKR
- removed U8: ACS706xLC-05C, symbol Sensor_Current:ACS706xLC-05C
- removed U9: ISO1042BQDWVQ1, symbol QRET_CANBUS:ISO1042BQDWVQ1
- added BZ2: PKM13EPYH4000, footprints:Buzzer_12.6x9.5RM5.0, symbol Device:Buzzer
- added C10: 10p, Capacitor_SMD:C_0603_1608Metric, symbol Device:C
- added C14: 100uF, Capacitor_SMD:CP_Elec_6.3x5.9, symbol Device:C_Polarized
- added C18: 0.1uF, Capacitor_SMD:C_0603_1608Metric, symbol Device:C
- added C2: 1uF, Capacitor_SMD:C_0603_1608Metric, symbol Device:C
- added C22, C23: 0.1u, Capacitor_SMD:C_0603_1608Metric, symbol Device:C
- added C30: 100nF, Capacitor_SMD:C_0603_1608Metric, symbol Device:C
- added C31, C32: 10uF, Capacitor_SMD:C_0603_1608Metric, symbol Device:C
- added D2: WS2812B, LED_SMD:LED_WS2812B_PLCC4_5.0x5.0mm_P3.2mm, symbol LED:WS2812B
- added D3: DB_LED (YLW), LED_SMD:LED_0603_1608Metric, symbol Device:LED
- added D5, D6: 1N5819WS, Diode_SMD:D_SOD-323, symbol Diode:1N5819WS
- added J1: Stack Male Edge Connector, Connector_PCBEdge:BUS_PCIexpress_x1, symbol EdgeConnector:Stack Male Edge Connector
- added J2: SWD_01x04_Pin, SWD_Header:SWD_PinHeader_1x04_P2.54mm_Horizontal, symbol EdgeConnector:SWD_01x04_Pin
- added J4: USB_B_Micro, footprints:USB_Micro-B_Amphenol_10118194_Horizontal, symbol Connector:USB_B_Micro
- added Q3: AO3400A, Package_TO_SOT_SMD:SOT-23, symbol Transistor_FET:AO3400A
- added R12, R13: 100k, Resistor_SMD:R_0603_1608Metric, symbol Device:R
- added R14: 510R, Resistor_SMD:R_0603_1608Metric, symbol Device:R
- added R15, R2, R4, R6: 10k, Resistor_SMD:R_0603_1608Metric, symbol Device:R
- added R16: 1k, Resistor_SMD:R_0603_1608Metric, symbol Device:R
- added R5: 820R, Resistor_SMD:R_0603_1608Metric, symbol Device:R
- added R7: 560R, Resistor_SMD:R_0603_1608Metric, symbol Device:R
- added R8: 1.5k, Resistor_SMD:R_0603_1608Metric, symbol Device:R
- added SW1: SW_STM_RESET, Button_Switch_SMD:SW_Push_1P1T_XKB_TS-1187A, symbol Switch:SW_Push
- added SW2: SW_STM_BOOT_MODE, Button_Switch_SMD:SW_Push_1P1T_XKB_TS-1187A, symbol Switch:SW_Push
- added TP2: TP_ISENSE, TestPoint:TestPoint_Pad_1.5x1.5mm, symbol Connector:TestPoint
- added TP3: TP_GND, TestPoint:TestPoint_Pad_1.5x1.5mm, symbol Connector:TestPoint
- added TP4: TP_3V3, TestPoint:TestPoint_Pad_1.5x1.5mm, symbol Connector:TestPoint
- added TP5: TP_VSTACK, TestPoint:TestPoint_Pad_1.5x1.5mm, symbol Connector:TestPoint
- added TP6: TP_VUSB, TestPoint:TestPoint_Pad_1.5x1.5mm, symbol Connector:TestPoint
- added TP7: TP_VSWD, TestPoint:TestPoint_Pad_1.5x1.5mm, symbol Connector:TestPoint
- added TP8: TP_MUX, TestPoint:TestPoint_Pad_1.5x1.5mm, symbol Connector:TestPoint
- added U1, U5, U6: LM66100DCKR, DCK6_TEX, symbol QRET_Buck_PSU-symbols:LM66100DCKR
- added U10: ACS70331EOLC, footprints:SOIC127P600X175-8N, symbol Sensor_Current:ACS706xLC-05C
- added U12: AMS1117-3.3, Package_TO_SOT_SMD:SOT-223-3_TabPin2, symbol Regulator_Linear:AMS1117-3.3
- added U3: W25Q128JVS, Package_SO:SOIC-8_5.23x5.23mm_P1.27mm, symbol Memory_Flash:W25Q128JVS
- added U8: ISO1042BDWVR, ISO1042:SOIC-8 ISO1042BDWV, symbol ISO1042BQDWVQ1:ISO1042BQDWVQ1
- C4: value 9p -> 1uF; footprint (none) -> Capacitor_SMD:C_0603_1608Metric; LCSC (none) -> C15849
- C6: value 1u -> 1uF; footprint (none) -> Capacitor_SMD:C_0603_1608Metric; LCSC (none) -> C15849
- C7: value 9p -> 10p; footprint (none) -> Capacitor_SMD:C_0603_1608Metric; LCSC (none) -> C1634
- C8: value 1u -> 100nF; footprint (none) -> Capacitor_SMD:C_0603_1608Metric; LCSC (none) -> C14663
- D1: value PWR_LED -> PWR_LED (GRN); footprint (none) -> LED_SMD:LED_0805_2012Metric; LCSC (none) -> C2297
- Y1: footprint (none) -> Crystal:Crystal_SMD_3225-4Pin_3.2x2.5mm; LCSC (none) -> C13738
Connections:
- net V_REG is gone; now on net +3.3V: C8.1
- net +3.3V: now also C22.2, D2.1 (VDD), D6.2 (A), J1.A1 (3.3V_A), J1.A2 (3.3V_A), R2.2, R4.2, R5.2, R6.2, R8.2, SW2.2, TP4.1, U10.3 (IP-), U10.4 (IP-), U3.8 (VCC), U8.1 (VCC1)
- net +5V: now also C23.2, J1.A4 (5.0V_A), J1.A5 (5.0V_A), U8.8 (VCC2)
- net BOOT0: now also R12.2, SW2.1
- net CAN_H: now also J1.B14 (CAN_H), U8.7 (CANH)
- net CAN_L: now also J1.B13 (CAN_L), U8.6 (CANL)
- net CAN_RX: now also U8.3 (RXD)
- net CAN_TX: now also U8.2 (TXD)
- net CS_FL: now also U3.1 (~{CS})
- net GND: now also C10.2, C14.2, C18.2, C2.2, C22.1, C23.1, C30.2, C31.2, C32.2, D2.3 (VSS), D3.1 (K), J1.A3 (GND_A), J1.A6 (GND_A), J1.B4 (GND_A), J1.B5 (GND_A), J1.B6 (GND_A), J2.1 (GND), J4.5 (GND), Q3.2 (S), R12.1, R13.1, R15.1, SW1.1, TP3.1, U1.2 (GND), U1.5 (ST), U10.5 (GND), U12.1 (GND), U3.4 (GND), U5.2 (GND), U5.5 (ST), U6.2 (GND), U6.5 (ST), U8.4 (GND1), U8.5 (GND2)
- net MISO_FL: now also U3.2 (DO(IO1))
- net MOSI_FL: now also U3.5 (DI(IO0))
- net OSC_IN: now also C7.1; no longer C4.1
- net OSC_OUT: now also C10.1; no longer C7.1
- net RESET_FL: now also R4.1, U3.7 (IO3)
- net SCK_FL: now also U3.6 (CLK)
- net SWCLK: now also J2.4 (SWCLK)
- net SWDIO: now also J2.3 (SWDIO)
- net V_PSU: now also C2.1, TP5.1, U1.1 (VIN)
- net V_SWD: now also J2.2 (3V3), TP7.1, U6.1 (VIN)
- net at D1.2 (A): now also R5.1
- net RGB: no longer names the net of D4.4 (DIN)
- net RGB: now also D2.2 (DOUT)
- new net: BZ2.1 (-), D5.1 (K), D6.1 (K), R16.2
- new net: BZ2.2 (+), Q3.3 (D), R16.1
- new net: R6.1, U3.3 (IO2)
- new net: D3.2 (A), R7.1
- new net: J1.A12 (GND_B), J1.A9 (GND_B), J1.B10 (GND_B), J1.B11 (GND_B), J1.B12 (GND_B)
- new net: J1.A7 (3.3V_B), J1.A8 (3.3V_B)
- new net: J1.B7 (BATT_B), J1.B8 (BATT_B), J1.B9 (BATT_B)
- new net: Q3.1 (G), R14.1
- new net +BATT: D5.2 (A), J1.B1 (BATT_A), J1.B2 (BATT_A), J1.B3 (BATT_A)
- new net BOOT1: R13.2
- new net BUZZER: R14.2, R15.2
- new net CURR_SENSE: TP2.1, U10.7 (VOUT)
- new net DB_LED: R7.2
- new net RGB_DATA: D2.4 (DIN)
- new net STM_RESET: C30.1, R2.1, SW1.2
- new net USB_5V: C31.1, J4.1 (VBUS), U12.3 (VI)
- new net USB_D+: J4.3 (D+), R8.1
- new net USB_D-: J4.2 (D-)
- new net V_MUX: C14.1, C18.1, TP8.1, U1.3 (*CE), U1.6 (VOUT), U10.1 (IP+), U10.2 (IP+), U10.8 (VCC), U5.3 (*CE), U5.6 (VOUT), U6.3 (*CE), U6.6 (VOUT)
- new net V_REGUSB: C32.1, C4.1, TP6.1, U12.2 (VO), U5.1 (VIN)
- no-connect marks 10 -> 9
Other:
- note added: "B0 HIGH = PROGRAMMING MODE B0 LOW = RUN MEMORY"
- note added: "CANBUS Interface"
- note added: "Current Sense & 3.3V Output"
- note added: "Flash Module (SPI)"
- note added: "Galvanic isolation barrier (we're not using isolation for primary modules)"
- note added: "Ideal Diodes (MUX)"
- note added: "Mount connector at edge of board"
- note added: "Put near edges of board (small & hard to solder)"
- note added: "RGB + Debug LEDs"
- note added: "STM32 Boot Mode"
- note added: "STM32 Reset"
- note added: "The WS2812B needs at least 3.5V input, but we're only using 3.3V This may cause problems"
- note added: "To Do: -Music -Light Sensor (LDR, photoresistor)"
- note added: "USB Connection"
- note added: "Vf=2.3V, I=1.8mA, R=560"
- note added: "Vf=2.9V, I=0.5mA, R=820"
- note added: "X322516MMB4SI Crystal"
- note added: "decoupling cap; place close to ACS70331"
- note removed: "-> go to connectors ->"
- note removed: "Also SPI no ic2"
- note removed: "Boot Mode"
- note removed: "CANBUS"
- note removed: "Current Sense + 3.3V output"
- note removed: "Flash Module"
- note removed: "Galvanic isolation barrier"
- note removed: "HIGH = PROGRAMMING MODE LOW = RUN MEMORY"
- note removed: "Ideal Diodes"
- note removed: "Need iso GND, and iso power supply VCC2 range: 4.5 > VCC2 > 5.5"
- note removed: "Put on one of the sides (really small and hard to soder)"
- note removed: "RGB Indicator"
- note removed: "ST pins are just status indication, Want a way to keep track of what power supply active?"
- note removed: "To Do: -Flash Module -Magnotometer -Music -Light Sensor (LDR, photoresistor) -Boot and Reset Buttons"
- note removed: "USB"
- note removed: "Units? (Capacitors) -ID"
- note removed: "can u use the same pullup?"
- note removed: "needed if same node as 1000u?"
- company: (none) -> Queen's Rocket Engineering Team
- moved on the sheet: C1, C11, C16, C17, C18, C20, C21, J4, J5, JP1, NAU1, R1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

Commit message: Various changes
It's been a while idk what these were lol
Parts:
- removed C1: 100n, symbol Device:C
- removed R1 (x2): 2.7k, symbol Device:R_US
- added C11: 10uF, Capacitor_SMD:CP_Elec_4x5.4, symbol Device:C_Polarized
- added C12, C13, C15, C17: 100n, Capacitor_SMD:C_0402_1005Metric, symbol Device:C
- added C19: 10n, Capacitor_SMD:C_0603_1608Metric, symbol Device:C
- added C20, C21: 1uF, Capacitor_SMD:C_0805_2012Metric, symbol Device:C_Polarized
- added FB1: 100R, Resistor_SMD:R_0805_2012Metric, symbol Device:FerriteBead
- added R1, R3: 4.7k, Resistor_SMD:R_0603_1608Metric, symbol Device:R
- added TP10: TP_SCL, TestPoint:TestPoint_Pad_1.5x1.5mm, symbol Connector:TestPoint
- added TP9: TP_SDA, TestPoint:TestPoint_Pad_1.5x1.5mm, symbol Connector:TestPoint
- added U9: BME680, Package_LGA:Bosch_LGA-8_3x3mm_P0.8mm_ClockwisePinNumbering, symbol Sensor:BME680
- C18: footprint Capacitor_SMD:C_0603_1608Metric -> Capacitor_SMD:C_0603_1608Metric_Pad1.08x0.95mm_HandSolder
- U4: LCSC (none) -> C404328
Connections:
- net D+ is gone; now on net USB_D+: U1.33 (PA12)
- net D- is gone; now on net USB_D-: U1.32 (PA11)
- net SDCLK is gone; now on net SWCLK: U1.37 (PA14)
- net V_BUZZ is gone; now on net BUZZER: U1.30 (PA9)
- net +3.3V: now also C11.1, C12.1, C13.1, C15.1, C17.1, C21.1, FB1.2, R1.2, R3.1
- net +3.3VA: now also C19.1, C20.1, FB1.1
- net BOOT1: now also U1.20 (PB2)
- net CURR_SENSE: now also U1.19 (PB1)
- net DB_LED: now also U1.38 (PA15)
- net GND: now also C11.2, U4.A1 (VSA), C11.2, C12.2, C13.2, C15.2, C17.2, C19.2, C20.2, C21.2
- net RGB_DATA: now also U1.39 (PB3)
- net STM_RESET: now also U1.7 (NRST)
- net SCL: now reaches U4.A2 (SCL)
- net SCL: now also U1.21 (PB10), R3.2, TP10.1
- net SDA: now reaches U4.B2 (SDA)
- net SDA: now also U1.22 (PB11), R1.1, TP9.1
- net V_Isense: no longer names the net of U1.10 (PA0)
- net V_MAG: no longer names the net of U1.41 (PB5)
- no-connect marks 9 -> 14
Other:
- note added: "Additional Filtering for Analogue VDD"
- note added: "Definitely add a "slot" for an expansion card"
- note added: "I2C ADDRESS: 0x30"
- note added: "ITS OUT OF STOCK ON JLCPCB DAMMIT BM1422AGMV-ZE2? Order of magnitude less sensitive Digikey?"
- note added: "Must be able to handle a 15V input (add slots for a voltage div)"
- note added: "One 100nf "high quality ceramic" capacitor for each VDD and VBAT One 10uf electrolytic capacitor for bulk filtering. Place them as close as possible to the IC - one cap per input pin"
- note added: "Remove ground plane beneath chip?"
- note added: "STM32 Decoupling Capacitors for VBAT and VDD"
- note added: "To Do: -Music -Light Sensor (LDR, photoresistor) -ADD BACK MCU DECOUPLING CAPS"
- note removed: "Be wary of the resistor count (depending on how many sensors)"
- note removed: "Capacitor to prevent unintended resets"
- note removed: "To Do: -Music -Light Sensor (LDR, photoresistor)"
- moved on the sheet: C11, U4

Commit message: Major updates
-Changed to USB C connector
-Added CP2102 USB-UART bridge
-Added RunCam control pins
-Added new magnetometer (BM1422AGMV)
-Added BME680 sensor
-Changed PWR LED resistor to 3.3k
Parts:
- removed C32: 10uF, Capacitor_SMD:C_0603_1608Metric, symbol Device:C
- removed J4: USB_B_Micro, footprints:USB_Micro-B_Amphenol_10118194_Horizontal, symbol Connector:USB_B_Micro
- added C28, C34, C35: 1uF, symbol Device:C
- added C3 (x2), C32: 10uF, Capacitor_SMD:C_0603_1608Metric, symbol Device:C
- added C3: 1uF, Capacitor_SMD:C_0603_1608Metric, symbol Device:C
- added C32, C33: 100nF, symbol Device:C
- added J4: USB_C_Female_USB2_Small, footprints:USB_C_DB-108PWB, symbol USB_C:USB_C_Female_USB2_Small
- added J6: CAM_PWR, TerminalBlock_TE-Connectivity:TerminalBlock_TE_282834-2_1x02_P2.54mm_Horizontal, symbol Connector:Screw_Terminal_01x02
- added J7: CAM_DAT, TerminalBlock_TE-Connectivity:TerminalBlock_TE_282834-3_1x03_P2.54mm_Horizontal, symbol Connector:Screw_Terminal_01x03
- added Q3: AO3401A, Package_TO_SOT_SMD:SOT-23, symbol Transistor_FET:AO3401A
- added Q4: AO3400A, Package_TO_SOT_SMD:SOT-23, symbol Transistor_FET:AO3400A
- added R10, R38: 100k, Resistor_SMD:R_0603_1608Metric, symbol Device:R
- added R28, R29: 5.1k, Resistor_SMD:R_0603_1608Metric, symbol Device:R
- added R29: 1k, Resistor_SMD:R_0603_1608Metric, symbol Device:R
- added R30: 22k, Resistor_SMD:R_0603_1608Metric, symbol Device:R
- added R31: 47k, Resistor_SMD:R_0603_1608Metric, symbol Device:R
- added R39: 510, Resistor_SMD:R_0603_1608Metric, symbol Device:R
- added TP13: TP_PA5, TestPoint:TestPoint_Pad_1.5x1.5mm, symbol Connector:TestPoint
- added TP14: TP_PA6, TestPoint:TestPoint_Pad_1.5x1.5mm, symbol Connector:TestPoint
- added TP15: TP_PA7, TestPoint:TestPoint_Pad_1.5x1.5mm, symbol Connector:TestPoint
- added U1: CP2102N-Axx-xQFN28, Package_DFN_QFN:QFN-28-1EP_5x5mm_P0.5mm_EP3.35x3.35mm, symbol Interface_USB:CP2102N-Axx-xQFN28
- added U12: BM1422AGMV, Package_LGA:Rohm_MLGA010V020A_LGA-10_2x2mm_P0.45mm_LayoutBorder_3x2y, symbol Sensor_Magnetic:BM1422AGMV
- C11, U4: now left out of the parts list
- R5: value 820R -> 3.3k; LCSC C23253 -> (none)
- U1: value STM32F103CBTx -> STM32F103CBT6; LCSC (none) -> C8304
Connections:
- net +3.3V: now also R8.1, U9.2 (CSB), U9.5 (SDO), U9.6 (VDDIO), U9.8 (VDD), C28.1, C3.2, C32.1, C33.1, C35.1, U1.6 (VDD), U1.7 (VREGIN), U12.1 (AVDD), U12.10 (DVDD); no longer R8.2
- net +5V: now also Q3.2 (S), R10.1
- net BUZZER: now also U1.17 (PA7); no longer U1.30 (PA9)
- net GND: now also U9.1 (GND), U9.7 (GND), C28.2, C3.1, C3.1, C3.2, C32.2, C32.2, C33.2, C34.2, C35.2, J4.A1 (GND), J4.A12 (GND), J4.B1 (GND), J4.B12 (GND), J6.1 (Pin_1), Q4.2 (S), R28.2, R29.2, R29.2, R31.1, R38.2, U1.29 (GND), U1.3 (GND), U12.2 (GND), U12.9 (ADDR)
- net SCL: now also U9.4 (SCK), U12.7 (SCL)
- net SDA: now also U9.3 (SDI), U12.5 (SDA)
- net USB_D+: now also R8.2, J4.A6 (D+), J4.B6 (D+), U1.4 (D+); no longer R8.1, U1.33 (PA12)
- net USB_D-: now also J4.A7 (D-), J4.B7 (D-), U1.5 (D-); no longer U1.32 (PA11)
- net V_REGUSB: now also C32.1
- net at U1.14 (PA4): now also TP13.1
- net at U1.15 (PA5): now also TP14.1
- net at U1.16 (PA6): now also TP15.1
- net CAM_RX: now reaches U1.31 (PA10)
- net CAM_RX: now also J7.3 (Pin_3)
- net USB_5V renamed 5V_RAW
- net 5V_RAW: now also J4.A4 (VBUS), J4.A9 (VBUS), J4.B4 (VBUS), J4.B9 (VBUS), R30.2
- net V_CLK: no longer names the net of NAU1.13 (SCLK)
- net V_CLK: no longer U1.13 (PA3)
- net V_DI: no longer names the net of U1.11 (PA1)
- net V_DI: no longer NAU1.14 (SDIO)
- net V_DR: no longer names the net of NAU1.12 (DRDY)
- net V_DR: no longer U1.12 (PA2)
- new net: J4.A5 (CC1), R29.1
- new net: J4.B5 (CC2), R28.1
- new net: C3.2, R30.1, R31.2, U1.8 (VBUS)
- new net: C34.1, U12.3 (VREG)
- new net: R29.1, U1.9 (~{RST})
- new net: Q3.1 (G), Q4.3 (D), R10.2
- new net: Q4.1 (G), R39.2
- new net CAM_5V: C3.1, J6.2 (Pin_2), Q3.3 (D)
- new net CAM_PWM: J7.1 (Pin_1), U1.32 (PA11)
- new net CAM_PWR: R38.1, R39.1
- new net CAM_TX: J7.2 (Pin_2), U1.30 (PA9)
- new net USB_RX: U1.13 (PA3), U1.26 (TXD)
- new net USB_TX: U1.12 (PA2), U1.25 (RXD)
- no-connect marks 14 -> 34
Other:
- note added: "BME680"
- note added: "I2C ADDRESS: 0x76 (SDO GND) >0x77 (SDO 3.3V)"
- note added: "I2C ADDRESS: >0x0E (ADDR = GND) 0X0F (ADDR = 3.3V)"
- note added: "Magnetometer (A)"
- note added: "Magnetometer (B)"
- note added: "RunCam Control"
- note added: "USB-UART Bridge"
- note added: "Vf=2.9V, I=????mA, R=3.3k"
- note removed: "Definitely add a "slot" for an expansion card"
- note removed: "ITS OUT OF STOCK ON JLCPCB DAMMIT BM1422AGMV-ZE2? Order of magnitude less sensitive Digikey?"
- note removed: "Magnetometer"
- note removed: "Maybe?"
- note removed: "To Do: -Music -Light Sensor (LDR, photoresistor) -ADD BACK MCU DECOUPLING CAPS"
- note removed: "Vf=2.9V, I=0.5mA, R=820"
- title: QRET 23-24 SRAD Sensors Module -> QRET 23-24 SRAD Sensors Module (COTIJA)
- moved on the sheet: C10, C11, C12, C13, C15, C16, C17, C18, C19, C20, C21, C30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
