File: Schematics/Sensors_Module/Sensors_Module.kicad_sch (KiCad schematic)
At the start: 98 parts, among them J1 Stack Male Edge Connector, J2 SWD_01x04_Pin, J4 USB_C_Female_USB2_Small, J6 CAM_PWR, J7 CAM_DAT, Q3 AO3400A, Q3 AO3401A, Q4 AO3400A, SW1 SW_STM_RESET, SW2 SW_STM_BOOT_MODE, U1 CP2102N-Axx-xQFN28, U1 LM66100DCKR, U1 STM32F103CBT6, U10 ACS70331EOLC, U12 AMS1117-3.3, U12 BM1422AGMV, U3 W25Q128JVS, U5 LM66100DCKR, U6 LM66100DCKR, U8 ISO1042BDWVR, U9 BME680, Y1 X322516MMB4SI

Commit message: Final tweaks
Connections:
- net D+ renamed CAN_H
- net D- renamed CAN_L
Changed lines of the file:
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@@
     )
   )
-  (global_label "D+" (shape bidirectional) (at 398.78 35.56 0) (fields_autoplaced)
-    (effects (font (size 1.27 1.27)) (justify left))
-    (property "Intersheetrefs" "${INTERSHEET_REFS}" (at 405.7189 35.56 0)
+  (global_label "CAN_H" (shape bidirectional) (at 398.78 35.56 0) (fields_autoplaced)
+    (effects (font (size 1.27 1.27)) (justify left))
+    (property "Intersheetrefs" "${INTERSHEET_REFS}" (at 408.8637 35.56 0)
       (effects (font (size 1.27 1.27)) (justify left) hide)
     )
@@
     )
   )
-  (global_label "D-" (shape bidirectional) (at 398.78 40.64 0) (fields_autoplaced)
-    (effects (font (size 1.27 1.27)) (justify left))
-    (property "Intersheetrefs" "${INTERSHEET_REFS}" (at 405.7189 40.64 0)
+  (global_label "CAN_L" (shape bidirectional) (at 398.78 40.64 0) (fields_autoplaced)
+    (effects (font (size 1.27 1.27)) (justify left))
+    (property "Intersheetrefs" "${INTERSHEET_REFS}" (at 408.5613 40.64 0)
       (effects (font (size 1.27 1.27)) (justify left) hide)
     )
@@
     )
   )
-  (global_label "D+" (shape input) (at 377.19 177.8 180) (fields_autoplaced)
-    (effects (font (size 1.27 1.27)) (justify right))
-    (property "Intersheetrefs" "${INTERSHEET_REFS}" (at 371.3624 177.8 0)
+  (global_label "CAN_H" (shape input) (at 377.19 177.8 180) (fields_autoplaced)
+    (effects (font (size 1.27 1.27)) (justify right))
+    (property "Intersheetrefs" "${INTERSHEET_REFS}" (at 368.2176 177.8 0)
       (effects (font (size 1.27 1.27)) (justify right) hide)
     )
@@
     )
   )
-  (global_label "D-" (shape input) (at 377.19 173.99 180) (fields_autoplaced)
-    (effects (font (size 1.27 1.27)) (justify right))
-    (property "Intersheetrefs" "${INTERSHEET_REFS}" (at 371.3624 173.99 0)
-      (effects (font (size 1.27 1.27)) (justify right) hide)
-    )
+  (global_label "CAN_L" (shape input) (at 377.19 173.99 180) (fields_autoplaced)
+    (effects (font (size 1.27 1.27)) (justify right))
+    (property "Intersheetrefs" "${INTERSHEET_REFS}" (at 368.52 173.99 0)
+      (effects (font (size 1.27 1.27)) (justify right) hide)
+    )

Commit message: Schematic clean-up (remove outdated parts)
- Removed old BME680 + Magnetometer sensors
- Removed ACS70331 current sensor
- Removed old RunCam6 driver circuitry
- Fixed NRST pullup resistor on CP2102
- Changed USB-C port to new one (C5178541)
- Changed SWD header to SMD version
- Added revised buzzer circuit
- Added some missing 3D models
- Changed "LCSC" fields to "JLCPCB"
Parts:
- removed BZ2: PKM13EPYH4000, footprints:Buzzer_12.6x9.5RM5.0, symbol Device:Buzzer
- removed C28, C34, C35: 1uF, Capacitor_SMD:C_0603_1608Metric, symbol Device:C
- removed C3: 10uF, Capacitor_SMD:C_0603_1608Metric, symbol Device:C
- removed C32, C33: 100nF, Capacitor_SMD:C_0603_1608Metric, symbol Device:C
- removed J6: CAM_PWR, TerminalBlock_TE-Connectivity:TerminalBlock_TE_282834-2_1x02_P2.54mm_Horizontal, symbol Connector:Screw_Terminal_01x02
- removed J7: CAM_DAT, TerminalBlock_TE-Connectivity:TerminalBlock_TE_282834-3_1x03_P2.54mm_Horizontal, symbol Connector:Screw_Terminal_01x03
- removed Q3: AO3401A, Package_TO_SOT_SMD:SOT-23, symbol Transistor_FET:AO3401A
- removed Q3, Q4: AO3400A, Package_TO_SOT_SMD:SOT-23, symbol Transistor_FET:AO3400A
- removed R1, R3: 4.7k, Resistor_SMD:R_0603_1608Metric, symbol Device:R
- removed R10, R38: 100k, Resistor_SMD:R_0603_1608Metric, symbol Device:R
- removed R14: 510R, Resistor_SMD:R_0603_1608Metric, symbol Device:R
- removed R15: 10k, Resistor_SMD:R_0603_1608Metric, symbol Device:R
- removed R16: 1k, Resistor_SMD:R_0603_1608Metric, symbol Device:R
- removed R39: 510, Resistor_SMD:R_0603_1608Metric, symbol Device:R
- removed TP10: TP_SCL, TestPoint:TestPoint_Pad_1.5x1.5mm, symbol Connector:TestPoint
- removed TP2: TP_ISENSE, TestPoint:TestPoint_Pad_1.5x1.5mm, symbol Connector:TestPoint
- removed TP8: TP_MUX, TestPoint:TestPoint_Pad_1.5x1.5mm, symbol Connector:TestPoint
- removed TP9: TP_SDA, TestPoint:TestPoint_Pad_1.5x1.5mm, symbol Connector:TestPoint
- removed U10: ACS70331EOLC, footprints:SOIC127P600X175-8N, symbol Sensor_Current:ACS706xLC-05C
- removed U12: BM1422AGMV, Package_LGA:Rohm_MLGA010V020A_LGA-10_2x2mm_P0.45mm_LayoutBorder_3x2y, symbol Sensor_Magnetic:BM1422AGMV
- removed U9: BME680, Package_LGA:Bosch_LGA-8_3x3mm_P0.8mm_ClockwisePinNumbering, symbol Sensor:BME680
- added BZ1: PS1240P02BT, footprints:Buzzer_12.6x9.5RM5.0, symbol Device:Buzzer
- added U10: TPM8837C-SO1R, footprints:SOP-8_TPK, symbol TPM8837C-SO1R:TPM8837C-SO1R
- C10, C7: JLCPCB (none) -> C1634; LCSC C1634 -> (none)
- C12, C13, C15, C17: JLCPCB (none) -> C1525; LCSC C1525 -> (none)
- C18: value 0.1uF -> 100nF; JLCPCB (none) -> C14663; LCSC C14663 -> (none)
- C19: JLCPCB (none) -> C57112; LCSC C57112 -> (none)
- C2, C3, C4, C6: JLCPCB (none) -> C15849; LCSC C15849 -> (none)
- C20, C21: JLCPCB (none) -> C28323; LCSC C28323 -> (none)
- C22, C23, C30, C8: JLCPCB (none) -> C14663; LCSC C14663 -> (none)
- C3, C31, C32: JLCPCB (none) -> C96446; LCSC C96446 -> (none)
- D1: JLCPCB (none) -> C2297; LCSC C2297 -> (none)
- D3: JLCPCB (none) -> C72038; LCSC C72038 -> (none)
- D5, D6: JLCPCB (none) -> C191023; LCSC C191023 -> (none)
- FB1: JLCPCB (none) -> C1015; LCSC C1015 -> (none)
- J2: footprint SWD_Header:SWD_PinHeader_1x04_P2.54mm_Horizontal -> SWD_Header:SWD_PinHeader_1x04_P2.54mm_Horizontal_SMD
- J4: JLCPCB (none) -> C5178541; LCSC C2936184 -> (none)
- R12, R13: JLCPCB (none) -> C25803; LCSC C25803 -> (none)
- R2, R4, R6: JLCPCB (none) -> C25804; LCSC C25804 -> (none)
- R28, R29: JLCPCB (none) -> C23186; LCSC C23186 -> (none)
- R29: JLCPCB (none) -> C21190; LCSC C21190 -> (none)
- R30: JLCPCB (none) -> C31850; LCSC C31850 -> (none)
- R31: JLCPCB (none) -> C25819; LCSC C25819 -> (none)
- R5: JLCPCB (none) -> C22978; LCSC C22978 -> (none)
- R7: JLCPCB (none) -> C23228; LCSC C23228 -> (none)
- R8: JLCPCB (none) -> C22843; LCSC C22843 -> (none)
- SW1, SW2: JLCPCB (none) -> C318884; LCSC C318884 -> (none)
- U1, U5, U6: JLCPCB (none) -> C2869734; LCSC C2869734 -> (none)
- U1: JLCPCB (none) -> C6568; LCSC C6568 -> (none)
- U1: JLCPCB (none) -> C8304; LCSC C8304 -> (none)
- U12: JLCPCB (none) -> C6186; LCSC C6186 -> (none)
- U3: JLCPCB (none) -> C97521; LCSC C97521 -> (none)
- U8: JLCPCB (none) -> C484409; LCSC C484409 -> (none)
- Y1: JLCPCB (none) -> C13738; LCSC C13738 -> (none)
Connections:
- net CAM_PWM is gone; now on net RESET_FL: U1.32 (PA11)
- net V_MUX is gone; now on net +3.3V: C14.1, C18.1, U1.3 (*CE), U1.6 (VOUT), U5.3 (*CE), U5.6 (VOUT), U6.3 (*CE), U6.6 (VOUT)
- net +3.3V: now also R29.2, U10.7 (NSLEEP), U10.8 (VCC)
- net GND: now also U10.4 (GND); no longer R29.2
- net RESET_FL: no longer U1.29 (PA8)
- net at D5.1 (K), D6.1 (K): now also U10.1 (VM)
- net BUZZER renamed BUZZER_A
- net BUZZER_A: now also U10.6 (IN1)
- net CAM_PWR: no longer names the net of U1.18 (PB0)
- net CAM_RX: no longer names the net of U1.31 (PA10)
- net CAM_TX: no longer names the net of U1.30 (PA9)
- net CURR_SENSE: no longer names the net of U1.19 (PB1)
- net SCL: no longer names the net of U1.21 (PB10)
- net SDA: no longer names the net of U1.22 (PB11)
- new net: BZ1.1 (-), U10.3 (OUT2)
- new net: BZ1.2 (+), U10.2 (OUT1)
- new net BUZZER_B: U1.29 (PA8), U10.5 (IN2)
- no-connect marks 31 -> 36
Other:
- note added: "Driving via 2 inverse PWM pins & H-Bridge to effectively double voltage across buzzer"
- note added: "Dual supply input so can test buzzer w/o battery present"
- note added: "Ideal Diodes (Input MUX + RPP)"
- note added: "Vf=2.8V, R=0.15mA, R=3.3k"
- note removed: "BME680"
- note removed: "I2C ADDRESS: 0x76 (SDO GND) >0x77 (SDO 3.3V)"
- note removed: "I2C ADDRESS: >0x0E (ADDR = GND) 0X0F (ADDR = 3.3V)"
- note removed: "Ideal Diodes (MUX)"
- note removed: "Magnetometer (B)"
- note removed: "Put near edges of board (small & hard to solder)"
- note removed: "Remove ground plane beneath chip?"
- note removed: "RunCam Control"
- note removed: "Vf=2.9V, I=????mA, R=3.3k"
- note removed: "decoupling cap; place close to ACS70331"
- moved on the sheet: C10, C14, C2, C3, C30, C31, C32, C4, C6, C7, D1, J1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

Commit message: Finished schematic
-Added ADS1256 ADCs
-Added analog voltage systems
-Added wheatstone bridge strain gauge circuits
-Added connectors
-Adjusted pinout
Parts:
- removed TP13: PB7, TestPoint:TestPoint_Pad_1.5x1.5mm, symbol Connector:TestPoint
- removed TP13: PB6, TestPoint:TestPoint_Pad_1.5x1.5mm, symbol Connector:TestPoint
- removed TP13: PA0, TestPoint:TestPoint_Pad_1.5x1.5mm, symbol Connector:TestPoint
- removed TP13: PA4, TestPoint:TestPoint_Pad_1.5x1.5mm, symbol Connector:TestPoint
- removed TP14: PA5, TestPoint:TestPoint_Pad_1.5x1.5mm, symbol Connector:TestPoint
- removed TP14: PB5, TestPoint:TestPoint_Pad_1.5x1.5mm, symbol Connector:TestPoint
- removed TP15: PA6, TestPoint:TestPoint_Pad_1.5x1.5mm, symbol Connector:TestPoint
- removed TP15: PB4, TestPoint:TestPoint_Pad_1.5x1.5mm, symbol Connector:TestPoint
- added C3: 1uF, Capacitor_SMD:C_0603_1608Metric, symbol Device:C
- added C31, C32 (x5): 10uF, Capacitor_SMD:C_0603_1608Metric, symbol Device:C
- added C44, C46, C48, C49, C52, C53, C54, C55: 100p, Capacitor_SMD:C_0402_1005Metric, symbol Device:C_Small
- added C45, C47, C50, C51, C56, C57, C58, C59: 0.1u, Capacitor_SMD:C_0603_1608Metric, symbol Device:C_Small
- added C46 (x9): 0.1u, Capacitor_SMD:C_0603_1608Metric, symbol Device:C
- added C46 (x4): 47uF, Capacitor_SMD:C_0805_2012Metric, symbol Device:C
- added C46 (x2): 100uF, Capacitor_SMD:C_1206_3216Metric, symbol Device:C
- added C46 (x2): 100p, Capacitor_SMD:C_0402_1005Metric, symbol Device:C
- added C46: 2.2uF, Capacitor_SMD:C_0603_1608Metric, symbol Device:C
- added C7 (x4): 20pF, Capacitor_SMD:C_0402_1005Metric, symbol Device:C
- added J10, J11, J12, J13, J14, J15, J4, J5, J6, J7, J8, J9: In, TerminalBlock_TE-Connectivity:TerminalBlock_TE_282834-2_1x02_P2.54mm_Horizontal, symbol Connector:Screw_Terminal_01x02
- added JP1: CH1_BR, Jumper:SolderJumper-3_P1.3mm_Bridged12_RoundedPad1.0x1.5mm, symbol Jumper:SolderJumper_3_Bridged12
- added JP2: CH2_BR, Jumper:SolderJumper-3_P1.3mm_Bridged12_RoundedPad1.0x1.5mm, symbol Jumper:SolderJumper_3_Bridged12
- added JP3: CH3_BR, Jumper:SolderJumper-3_P1.3mm_Bridged12_RoundedPad1.0x1.5mm, symbol Jumper:SolderJumper_3_Bridged12
- added JP4: CH4_BR, Jumper:SolderJumper-3_P1.3mm_Bridged12_RoundedPad1.0x1.5mm, symbol Jumper:SolderJumper_3_Bridged12
- added JP5: CH5_BR, Jumper:SolderJumper-3_P1.3mm_Bridged12_RoundedPad1.0x1.5mm, symbol Jumper:SolderJumper_3_Bridged12
- added JP6: CH6_BR, Jumper:SolderJumper-3_P1.3mm_Bridged12_RoundedPad1.0x1.5mm, symbol Jumper:SolderJumper_3_Bridged12
- added JP7: CH7_BR, Jumper:SolderJumper-3_P1.3mm_Bridged12_RoundedPad1.0x1.5mm, symbol Jumper:SolderJumper_3_Bridged12
- added JP8: CH8_BR, Jumper:SolderJumper-3_P1.3mm_Bridged12_RoundedPad1.0x1.5mm, symbol Jumper:SolderJumper_3_Bridged12
- added Q1: AO3400A, Package_TO_SOT_SMD:SOT-23, symbol Transistor_FET:AO3400A
- added R17: 100k, Resistor_SMD:R_0603_1608Metric, symbol Device:R
- added R18: 510R, Resistor_SMD:R_0603_1608Metric, symbol Device:R
- added R4 (x4): 49.9R, Resistor_SMD:R_0402_1005Metric, symbol Device:R
- added R4 (x16): 330R, Resistor_SMD:R_0402_1005Metric, symbol Device:R
- added R4 (x6): 100R, Resistor_SMD:R_0402_1005Metric, symbol Device:R
- added R4 (x4): 10k, Resistor_SMD:R_0603_1608Metric, symbol Device:R
- added R7 (x16): 350R, Resistor_SMD:R_0805_2012Metric_Pad1.20x1.40mm_HandSolder, symbol Device:R
- added R7 (x8): 350, Resistor_SMD:R_0805_2012Metric_Pad1.20x1.40mm_HandSolder, symbol Device:R
- added TH1: 10k, Resistor_SMD:R_0603_1608Metric_Pad0.98x0.95mm_HandSolder, symbol Device:Thermistor_NTC
- added TP13: PB10, TestPoint:TestPoint_Pad_1.5x1.5mm, symbol Connector:TestPoint
- added TP13: PB0, TestPoint:TestPoint_Pad_1.5x1.5mm, symbol Connector:TestPoint
- added U12, U4: ADS1256IDBR, footprints:SOP65P780X200-28N, symbol ADS1256IDBR:ADS1256IDBR
- added U13: OPA2727AIDR, footprints:SOIC127P599X175-8N-OPA2727, symbol OPA2727AIDR:OPA2727AIDR
- added U14: MCP1501-25xCH, Package_TO_SOT_SMD:SOT-23-6_Handsoldering, symbol Reference_Voltage:MCP1501-25xCH
- added U9: AMS1117-5.0, Package_TO_SOT_SMD:SOT-223-3_TabPin2, symbol Regulator_Linear:AMS1117-5.0
- added Y2, Y3: X50328MSB2GI, footprints:CRYSTAL-SMD_L5.0-W3.2, symbol Device:Crystal
- J2: Digikey (none) -> 952-3233-ND
Connections:
- net +3.3V: now also C32.1, C32.1, C46.1, C46.1, R4.1, R4.1, R4.2, U12.16 (DVDD), U4.16 (DVDD)
- net +BATT: now also C31.1, U9.3 (VI)
- net BUZZER_A: now also U1.31 (PA10); no longer U1.17 (PA7)
- net BUZZER_B: now also U1.19 (PB1); no longer U1.29 (PA8)
- net GND: now also C3.1, C31.2, C32.2, C32.2, C32.2, C32.2, C32.2, C46.1, C46.2, C46.2, C46.2, C46.2, C46.2, C46.2, C46.2, C46.2, C46.2, C46.2, C46.2, C7.1, C7.1, C7.2, C7.2, Q1.2 (S), R17.1, R4.1, R4.1, TH1.2, U12.17 (DGND), U12.2 (AGND), U12.5 (AINCOM), U13.4 (V-), U14.2 (GND), U14.3 (GND), U14.5 (GND), U4.17 (DGND), U4.2 (AGND), U4.5 (AINCOM), U9.1 (GND)
- net ADS_SYNC: now reaches U1.43 (PB7)
- net ADS_SYNC: now also R4.1, U12.14 (~{SYNC},_~{PDWN}), U4.14 (~{SYNC},_~{PDWN})
- net ADS_RESET: now reaches U1.42 (PB6)
- net ADS_RESET: now also R4.2, U12.15 (~{RESET}), U4.15 (~{RESET})
- net ADS_DOUT: now reaches U1.16 (PA6)
- net ADS_DOUT: now also U12.22 (DOUT), U4.22 (DOUT)
- net TEMP: now reaches U1.10 (PA0)
- net TEMP: now also R4.2, TH1.1
- net ADS1_CS: now reaches U1.14 (PA4)
- net ADS1_CS: now also R4.1
- net ADS_SCLK: now reaches U1.15 (PA5)
- net ADS_SCLK: now also R4.1, R4.1
- net at U1.18 (PB0): now also TP13.1
- net at U1.21 (PB10): now also TP13.1
- net WS_EN: now reaches U1.22 (PB11)
- net WS_EN: now also R17.2, R18.1
- net ADS1_DRDY: now reaches U1.40 (PB4)
- net ADS1_DRDY: now also U4.21 (~{DRDY})
- net ADS2_DRDY: now reaches U1.41 (PB5)
- net ADS2_DRDY: now also U12.21 (~{DRDY})
- new net: C52.1, C56.1, R4.2, U12.6 (AIN0)
- new net: C52.2, C56.2, R4.2, U12.7 (AIN1)
- new net: C46.2, C46.2, C46.2, R4.1, U12.4 (VREFP)
- new net: C48.2, C50.2, R4.2, U4.11 (AIN5)
- new net: C54.1, C58.1, R4.2, U12.10 (AIN4)
- new net: C55.1, C59.1, R4.2, U12.12 (AIN6)
- new net: C55.2, C59.2, R4.2, U12.13 (AIN7)
- new net: R4.2, U14.1 (OUT)
- new net: C46.1, C46.1, C46.1, R4.2, U12.3 (VREFN)
- new net: C54.2, C58.2, R4.2, U12.11 (AIN5)
- new net: JP7.1 (A), R7.2
- new net: C49.2, C51.2, R4.2, U4.13 (AIN7)
- new net: C46.2, C47.2, R4.2, U4.9 (AIN3)
- new net: JP4.1 (A), R7.2
- new net: JP3.1 (A), R7.2
- new net: JP6.1 (A), R7.2
- new net: C49.1, C51.1, R4.2, U4.12 (AIN6)
- new net: JP8.1 (A), R7.2
- new net: JP5.1 (A), R7.2
- new net: C46.1, C46.1, C46.1, R4.2, U4.3 (VREFN)
- new net: C46.2, C46.2, C46.2, R4.1, U4.4 (VREFP)
- new net: C48.1, C50.1, R4.2, U4.10 (AIN4)
- new net: R4.2, U4.20 (~{CS})
- new net: R4.2, U4.23 (DIN)
- new net: R4.2, U4.24 (SCLK)
- new net: C44.1, C45.1, R4.2, U4.6 (AIN0)
- new net: C44.2, C45.2, R4.2, U4.7 (AIN1)
- new net: C46.1, C47.1, R4.2, U4.8 (AIN2)
- new net: C3.2, R4.1, U13.3 (+IN_A), U13.5 (+IN_B)
- new net: C53.1, C57.1, R4.2, U12.8 (AIN2)
- new net: R4.2, U12.23 (DIN)
- new net: JP2.1 (A), R7.2
- new net: C53.2, C57.2, R4.2, U12.9 (AIN3)
- new net: JP1.1 (A), R7.2
- new net: Q1.1 (G), R18.2
- new net: R4.2, U12.20 (~{CS})
- new net: R4.2, U12.24 (SCLK)
- new net +5VA: C32.1, C32.1, C32.1, C46.1, C46.1, C46.1, C46.2, U12.1 (AVDD), U13.8 (V+), U14.4 (~{SHDN}), U14.6 (VDD), U4.1 (AVDD), U9.2 (VO)
- new net 2.5VA_1: C46.1, C46.1, C46.1, J4.1 (Pin_1), J5.2 (Pin_2), J7.1 (Pin_1), J8.2 (Pin_2), R4.2, R7.1, R7.1, R7.1, R7.1, U13.1 (OUT_A), U13.2 (-IN_A)
- new net 2.5VA_2: C46.1, C46.1, C46.1, J10.1 (Pin_1), J11.2 (Pin_2), J13.1 (Pin_1), J14.2 (Pin_2), R4.2, R7.1, R7.1, R7.1, R7.1, U13.6 (-IN_B), U13.7 (OUT_B)
- new net ADC1_X_IN: C7.2, U4.19 (XTAL1/CLKIN), Y2.2
- new net ADC1_X_OUT: C7.1, U4.18 (XTAL2), Y2.1
- new net ADC2_X_IN: C7.2, U12.19 (XTAL1/CLKIN), Y3.2
- new net ADC2_X_OUT: C7.1, U12.18 (XTAL2), Y3.1
- new net ADS2_CS: R4.1, U1.29 (PA8)
- new net ADS_DIN: R4.1, R4.1, U1.17 (PA7)
- new net CH1_L: J5.1 (Pin_1), JP1.3 (B)
- new net CH1_N: R4.1, R7.1, R7.2
- new net CH1_P: J4.2 (Pin_2), R4.1, R7.1
- new net CH2_L: J6.2 (Pin_2), JP2.3 (B)
- new net CH2_N: R4.1, R7.1, R7.2
- new net CH2_P: J6.1 (Pin_1), R4.1, R7.1
- new net CH3_L: J8.1 (Pin_1), JP3.3 (B)
- new net CH3_N: R4.1, R7.1, R7.2
- new net CH3_P: J7.2 (Pin_2), R4.1, R7.1
- new net CH4_L: J9.2 (Pin_2), JP4.3 (B)
- new net CH4_N: R4.1, R7.1, R7.2
- new net CH4_P: J9.1 (Pin_1), R4.1, R7.1
- new net CH5_L: J11.1 (Pin_1), JP5.3 (B)
- new net CH5_N: R4.1, R7.1, R7.2
- new net CH5_P: J10.2 (Pin_2), R4.1, R7.1
- new net CH6_L: J12.2 (Pin_2), JP6.3 (B)
- new net CH6_N: R4.1, R7.1, R7.2
- new net CH6_P: J12.1 (Pin_1), R4.1, R7.1
- new net CH7_L: J14.1 (Pin_1), JP7.3 (B)
- new net CH7_N: R4.1, R7.1, R7.2
- new net CH7_P: J13.2 (Pin_2), R4.1, R7.1
- new net CH8_L: J15.2 (Pin_2), JP8.3 (B)
- new net CH8_N: R4.1, R7.1, R7.2
- new net CH8_P: J15.1 (Pin_1), R4.1, R7.1
- new net GND_WS: JP1.2 (C), JP2.2 (C), JP3.2 (C), JP4.2 (C), JP5.2 (C), JP6.2 (C), JP7.2 (C), JP8.2 (C), Q1.3 (D), R7.2, R7.2, R7.2, R7.2, R7.2, R7.2, R7.2, R7.2
- no-connect marks 36 -> 39
Other:
- note added: "(its cheaper to get 12x 02 pin headers than 4x 06, 3x 08, etc)"
- note added: "* = Remap"
- note added: "ACS1256 draws ~50mA max on AVDD. 8x 350R wheatstone bridges @ 2.5V draw ~60mA. So ~160mA total."
- note added: "ADC 2.5V Analog Voltage Reference"
- note added: "ADC 5V Analog Power Source"
- note added: "ADC1 ADS1256"
- note added: "ADC1 Crystal Oscillator (8MHz)"
- note added: "ADC12_IN0"
- note added: "ADC2 ADS1256"
- note added: "ADC2 Crystal Oscillator (8MHz)"
- note added: "AMS1117-5.0: - Current: 1000mA (1.2VDO) - Accuracy: 2% (4.900V - 5.100V) - Regulation: 0.2% line, 0.4% load"
- note added: "AO3400A: - 0.048 ohm MAX Rds(on) - ~0.01% of 350R"
- note added: "Analog Power Source Temp Sensor"
- note added: "CANRX*"
- note added: "CANTX*"
- note added: "MCP1501-25x: - 2.5V ±0.1% - 20mA output max"
- note added: "MOST OF SCHEMATIC IS UP THERE /\"
- note added: "NOTE: JPx *MUST* BE SWITCHED IF CHx_L INPUT IS TO BE USED"
- note added: "OPA2727 Dual Buffer: - 40mA max out per chn. - 150µV max input offset"
- note added: "SPI1_MISO"
- note added: "SPI1_MOSI"
- note added: "SPI1_NSS (softNSS mngmnt)"
- note added: "SPI1_SCK"
- note added: "SPI2_MISO"
- note added: "SPI2_MOSI"
- note added: "SPI2_NSS"
- note added: "SPI2_SCK"
- note added: "STM32 Crystal Oscillator"
- note added: "Strain Gauge Inputs"
- note added: "TIM1_CH3"
- note added: "TIM1_CH3N*"
- note added: "USART2_RX"
- note added: "USART2_TX"
- note added: "Upper1 Common1 Lower1"
- note added: "Upper2 Common2 Lower2"
- note added: "Upper3 Common3 Lower3"
- note added: "Upper4 Common4 Lower4"
- note added: "Upper5 Common5 Lower5"
- note added: "Upper6 Common6 Lower6"
- note added: "Wheatstone Bridges (350±0.1%)"
- note added: "Wheatstone Shutoff"
- note removed: "Crystal Oscillator"
- moved on the sheet: TP14, U1

Commit message: Completed PCB layout
Wow that was disgusting
Parts:
- removed TP13: PB10, TestPoint:TestPoint_Pad_1.5x1.5mm, symbol Connector:TestPoint
- removed TP13: PB0, TestPoint:TestPoint_Pad_1.5x1.5mm, symbol Connector:TestPoint
- removed TP6: TP_VUSB, TestPoint:TestPoint_Pad_1.5x1.5mm, symbol Connector:TestPoint
- removed TP7: TP_VSWD, TestPoint:TestPoint_Pad_1.5x1.5mm, symbol Connector:TestPoint
- added Q2, Q3: AO3401A, Package_TO_SOT_SMD:SOT-23, symbol Transistor_FET:AO3401A
- added R17 (x2): 100k, Resistor_SMD:R_0402_1005Metric, symbol Device:R
- C32: footprint Capacitor_SMD:C_0603_1608Metric -> Capacitor_SMD:C_0402_1005Metric; JLCPCB C96446 -> C15525
- C46: value 0.1u -> 100n; footprint Capacitor_SMD:C_0603_1608Metric -> Capacitor_SMD:C_0402_1005Metric; JLCPCB C14663 -> C1525
- JP1, JP2, JP3, JP4, JP5, JP6, JP7, JP8: footprint Jumper:SolderJumper-3_P1.3mm_Bridged12_RoundedPad1.0x1.5mm -> Jumper:SolderJumper-3_P1.3mm_Open_RoundedPad1.0x1.5mm
- TP14: value PA1 -> PB11
- TP3: value TP_GND -> GND
- TP4: value TP_3V3 -> 3v3
- TP5: value TP_VSTACK -> VSTAK
Connections:
- net 2.5VA_1: now also C46.1, C46.1, C46.1, U13.6 (-IN_B), U13.7 (OUT_B), Q2.2 (S), R17.1; no longer C46.1, C46.1, C46.1, J4.1 (Pin_1), J5.2 (Pin_2), J7.1 (Pin_1), J8.2 (Pin_2), R7.1, R7.1, R7.1, R7.1, U13.1 (OUT_A), U13.2 (-IN_A)
- net 2.5VA_2: now also C46.1, C46.1, C46.1, U13.1 (OUT_A), U13.2 (-IN_A), Q3.2 (S), R17.1; no longer C46.1, C46.1, C46.1, J10.1 (Pin_1), J11.2 (Pin_2), J13.1 (Pin_1), J14.2 (Pin_2), R7.1, R7.1, R7.1, R7.1, U13.6 (-IN_B), U13.7 (OUT_B)
- net ADS1_DRDY: now also U1.21 (PB10); no longer U1.40 (PB4)
- net ADS2_CS: now also U1.39 (PB3); no longer U1.29 (PA8)
- net ADS2_DRDY: now also U1.40 (PB4); no longer U1.41 (PB5)
- net ADS_SYNC: now also U1.41 (PB5); no longer U1.43 (PB7)
- net CH1_L: now also J9.2 (Pin_2); no longer J5.1 (Pin_1)
- net CH1_P: now also J9.1 (Pin_1); no longer J4.2 (Pin_2)
- net CH2_L: now also J5.1 (Pin_1); no longer J6.2 (Pin_2)
- net CH2_P: now also J4.2 (Pin_2); no longer J6.1 (Pin_1)
- net CH4_L: now also J6.2 (Pin_2); no longer J9.2 (Pin_2)
- net CH4_P: now also J6.1 (Pin_1); no longer J9.1 (Pin_1)
- net CH5_L: now also J15.2 (Pin_2); no longer J11.1 (Pin_1)
- net CH5_P: now also J15.1 (Pin_1); no longer J10.2 (Pin_2)
- net CH6_L: now also J11.1 (Pin_1); no longer J12.2 (Pin_2)
- net CH6_P: now also J10.2 (Pin_2); no longer J12.1 (Pin_1)
- net CH8_L: now also J12.2 (Pin_2); no longer J15.2 (Pin_2)
- net CH8_P: now also J12.1 (Pin_1); no longer J15.1 (Pin_1)
- net DB_LED: now also D3.2 (A); no longer R7.2
- net GND: now also JP1.2 (C), JP2.2 (C), JP3.2 (C), JP4.2 (C), JP5.2 (C), JP6.2 (C), JP7.2 (C), JP8.2 (C), R7.1, R7.2, R7.2, R7.2, R7.2, R7.2, R7.2, R7.2, R7.2; no longer D3.1 (K)
- net RGB_DATA: now also U1.43 (PB7); no longer U1.39 (PB3)
- net WS_EN: now also R18.2, U1.11 (PA1); no longer R18.1, U1.22 (PB11)
- net ADC0B: now reaches C52.1, C56.1, R4.2, U12.6 (AIN0)
- net ADC1B: now reaches C52.2, C56.2, R4.2, U12.7 (AIN1)
- net ADC5A: now reaches C48.2, C50.2, R4.2, U4.11 (AIN5)
- net ADC4B: now reaches C54.1, C58.1, R4.2, U12.10 (AIN4)
- net ADC6B: now reaches C55.1, C59.1, R4.2, U12.12 (AIN6)
- net ADC7B: now reaches C55.2, C59.2, R4.2, U12.13 (AIN7)
- net ADC5B: now reaches C54.2, C58.2, R4.2, U12.11 (AIN5)
- net ADC7A: now reaches C49.2, C51.2, R4.2, U4.13 (AIN7)
- net ADC3A: now reaches C46.2, C47.2, R4.2, U4.9 (AIN3)
- net ADC6A: now reaches C49.1, C51.1, R4.2, U4.12 (AIN6)
- net ADC4A: now reaches C48.1, C50.1, R4.2, U4.10 (AIN4)
- net ADC0A: now reaches C44.1, C45.1, R4.2, U4.6 (AIN0)
- net ADC1A: now reaches C44.2, C45.2, R4.2, U4.7 (AIN1)
- net ADC2A: now reaches C46.1, C47.1, R4.2, U4.8 (AIN2)
- net ADC2B: now reaches C53.1, C57.1, R4.2, U12.8 (AIN2)
- net ADC3B: now reaches C53.2, C57.2, R4.2, U12.9 (AIN3)
- net at Q1.1 (G): now also R18.1; no longer R18.2
- net at TP14.1: now also U1.22 (PB11); no longer U1.11 (PA1)
- removed net GND_WS: JP1.2 (C), JP2.2 (C), JP3.2 (C), JP4.2 (C), JP5.2 (C), JP6.2 (C), JP7.2 (C), JP8.2 (C), Q1.3 (D), R7.2, R7.2, R7.2, R7.2, R7.2, R7.2, R7.2, R7.2
- new net: D3.1 (K), R7.2
- new net: Q1.3 (D), Q2.1 (G), Q3.1 (G), R17.2, R17.2
- new net 2.5VA_WS_1: J4.1 (Pin_1), J5.2 (Pin_2), J7.1 (Pin_1), J8.2 (Pin_2), Q2.3 (D), R7.1, R7.1, R7.1, R7.1
- new net 2.5VA_WS_2: J10.1 (Pin_1), J11.2 (Pin_2), J13.1 (Pin_1), J14.2 (Pin_2), Q3.3 (D), R7.1, R7.1, R7.1, R7.1
- no-connect marks 39 -> 41
Other:
- note added: "AO3401A: - 0.060 ohm TYP Rds(on) - ~0.017% of 350R"
- note added: "Technically this circuit couples 2.5VA_1 and 2.5VA_2 via a 200k resistor. This should have minimal impact."
- note removed: "AO3400A: - 0.048 ohm MAX Rds(on) - ~0.01% of 350R"
- moved on the sheet: D3, Q1, R17, R18, R7, TP14
