File: Schematics/Power_Module/Power_Module.kicad_pcb (KiCad board)
At the start: 4 copper layers, 69.5 x 60 mm, 50 parts, among them J1 ScrewSwitch A, J2 ScrewSwitch B, J3 Battery B, J5 Battery A, J6 Stack Male Edge Connector, Q1 AO4447A, Q2 AO4447A, U1 LMR51430XDDCR, U2 LMR51430XDDCR, U3 LMR51430XDDCR

Commit message: Revision bump to V2.0
Changed to V2.0 due to significant hardware changes
Other:
- board text added: "Halloumi Rev 2.0 QRET Feb 2025 Rajan Laird Kennan Bays Oak Campbell"
- board text removed: "Halloumi Rev 1.0 QRET Mar 2024 Rajan Laird Kennan Bays Oak Campbell"
Changed lines of the file:
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@@
   (gr_line (start 150.25 45.55) (end 150.25 39.75)
     (stroke (width 0.1) (type default)) (layer "Edge.Cuts"))
-  (gr_text "Halloumi Rev 1.0\nQRET Mar 2024\n\nRajan Laird\nKennan Bays\nOak Campbell" (at 165 50.9) (layer "B.SilkS")
+  (gr_text "Halloumi Rev 2.0\nQRET Feb 2025\n\nRajan Laird\nKennan Bays\nOak Campbell" (at 165 50.9) (layer "B.SilkS")
     (effects (font (size 1.5 1.5) (thickness 0.25)) (justify top mirror))
   )
