File: Schematics/Power_Module/Power_Module.kicad_pcb (KiCad board)
At the start: 4 copper layers, 69.5 x 60 mm, 131 parts, among them J1 ScrewSwitch B, J2 ScrewSwitch A, J3 Battery A, J4 USB_C_Female_USB2_Small, J5 Battery B, J6 Stack Male Edge Connector, J7 SWD_B, J8 SWD_B, Q1 AO4447A, Q2 AO4447A, U1 LMR51430XDDCR, U10 ISO1042BDWVR, U11 LM66100DCKR, U12 LM66100DCKR, U13 LM66100DCKR, U14 LM66100DCKR, U15 LM66100DCKR, U16 SCM3721ASA, U2 LMR51430XDDCR, U3 LMR51430XDDCR, U4 STM32F103C8T6, U5 STM32F103C8T6, U6 ACS37041KLHBLT-010B3, U7 ACS37041KLHBLT-010B3, U8 ACS37041KLHBLT-010B3, U9 AMS1117-3.3, Y1 X322516MMB4SI

Commit message: Final silkscreen tweak
Other:
- board text added: "LEVULOSE"
- board text added: "Power Module Rev 2.0 QRET Mar 2025 Rajan Laird Kennan Bays Oak Campbell"
- board text added: "Power Module V2.0"
- board text removed: "HALLOUMI V2.0"
- board text removed: "Halloumi Rev 2.0 QRET Feb 2025 Rajan Laird Kennan Bays Oak Campbell"
- board text removed: "Most annoying PCB we've made to date"
- board text removed: "Power Module"
Changed lines of the file:
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@@
       (plot_on_all_layers_selection 0x0000000_00000000)
       (disableapertmacros false)
-      (usegerberextensions false)
-      (usegerberattributes true)
-      (usegerberadvancedattributes true)
-      (creategerberjobfile true)
+      (usegerberextensions true)
+      (usegerberattributes false)
+      (usegerberadvancedattributes false)
+      (creategerberjobfile false)
       (dashed_line_dash_ratio 12.000000)
       (dashed_line_gap_ratio 3.000000)
@@
       (plotinvisibletext false)
       (sketchpadsonfab false)
-      (subtractmaskfromsilk false)
+      (subtractmaskfromsilk true)
       (outputformat 1)
       (mirror false)
-      (drillshape 1)
+      (drillshape 0)
       (scaleselection 1)
-      (outputdirectory "")
+      (outputdirectory "gerbers/")
     )
   )
@@
     (fp_line (start 1 0.625) (end -1 0.625)
       (stroke (width 0.1) (type solid)) (layer "F.Fab"))
-    (pad "1" smd roundrect (at -0.9125 0 90) (size 1.025 1.4) (layers "F.Cu" "F.Paste" "F.Mask") (roundrect_rratio 0.243902)
+    (pad "1" smd roundrect (at -0.9125 0 90) (size 1.025 1.4) (layers "F.Cu" "F.Paste" "F.Mask") (roundrect_rratio 0.243902439)
       (net 64 "3.3VA_B") (pintype "passive"))
-    (pad "2" smd roundrect (at 0.9125 0 90) (size 1.025 1.4) (layers "F.Cu" "F.Paste" "F.Mask") (roundrect_rratio 0.243902)
+    (pad "2" smd roundrect (at 0.9125 0 90) (size 1.025 1.4) (layers "F.Cu" "F.Paste" "F.Mask") (roundrect_rratio 0.243902439)
       (net 62 "V_MUX_B") (pintype "passive"))
     (model "${KICAD6_3DMODEL_DIR}/Resistor_SMD.3dshapes/R_0805_2012Metric.wrl"
@@
     (fp_line (start 1 0.625) (end -1 0.625)
       (stroke (width 0.1) (type solid)) (layer "F.Fab"))
-    (pad "1" smd roundrect (at -0.9125 0 90) (size 1.025 1.4) (layers "F.Cu" "F.Paste" "F.Mask") (roundrect_rratio 0.243902)
+    (pad "1" smd roundrect (at -0.9125 0 90) (size 1.025 1.4) (layers "F.Cu" "F.Paste" "F.Mask") (roundrect_rratio 0.243902439)
       (net 63 "3.3VA_A") (pintype "passive"))
-    (pad "2" smd roundrect (at 0.9125 0 90) (size 1.025 1.4) (layers "F.Cu" "F.Paste" "F.Mask") (roundrect_rratio 0.243902)
+    (pad "2" smd roundrect (at 0.9125 0 90) (size 1.025 1.4) (layers "F.Cu" "F.Paste" "F.Mask") (roundrect_rratio 0.243902439)
       (net 48 "V_MUX_A") (pintype "passive"))
     (model "${KICAD6_3DMODEL_DIR}/Resistor_SMD.3dshapes/R_0805_2012Metric.wrl"
@@
     (effects (font (size 1.3 1.3) (thickness 0.25) bold) (justify bottom mirror))
   )
-  (gr_text "Halloumi Rev 2.0\nQRET Feb 2025\n\nRajan Laird\nKennan Bays\nOak Campbell" (at 165 46.7) (layer "B.SilkS")
+  (gr_text "Power Module Rev 2.0\nQRET Mar 2025\n\nRajan Laird\nKennan Bays\nOak Campbell" (at 165 46.7) (layer "B.SilkS")
     (effects (font (size 1.5 1.5) (thickness 0.25)) (justify top mirror))
   )
@@
     (effects (font (size 1.4 1.4) (thickness 0.25) bold) (justify right bottom))
   )
-  (gr_text "HALLOUMI V2.0" (at 133.05 95.749998 90) (layer "F.SilkS" knockout)
+  (gr_text "LEVULOSE" (at 133.05 95.749998 90) (layer "F.SilkS" knockout)
     (effects (font (size 1.5 1.5) (thickness 0.3) bold) (justify left bottom))
   )
@@
     (effects (font (size 1.2 1.2) (thickness 0.15)) (justify bottom))
   )
-  (gr_text "Power Module" (at 135.6 95.749998 90) (layer "F.SilkS" knockout)
+  (gr_text "Power Module V2.0" (at 135.6 95.749998 90) (layer "F.SilkS" knockout)
     (effects (font (size 1.5 1.5) (thickness 0.3) bold) (justify left bottom))
   )
@@
     (effects (font (size 1 1) (thickness 0.15)) (justify left bottom))
   )
-  (gr_text "Most annoying PCB\nwe've made to date" (at 104.7 88) (layer "Cmts.User")
-    (effects (font (size 1 1) (thickness 0.15)) (justify left bottom))
-  )
