File: Schematics/Altimeter_Module/Altimeter_Module.kicad_sch (KiCad schematic)
At the start: 107 parts, among them J1 Stack Male Edge Connector, J2 Main E-Match, J3 Drogue E-Match, J4 USB_C_Female_USB2_Small, J5 SWD_01x04_Pin, Q1 AO3400A, Q2 AO4406AL, Q4 AO3400A, Q5 AO4406AL, SW1 SW_STM_RESET, SW2 SW_STM_BOOT_MODE, U1 QMA6100P, U10 TPM8837C-SO1R, U11 CP2102N-Axx-xQFN28, U12 AMS1117-3.3, U2 MS560702BA03-50, U3 W25Q128JVS, U4 LM66100DCKR, U5 LM66100DCKR, U6 STM32F103CBT6, U7 LM66100DCKR, U8 ISO1042BDWVR, U9 MPU-6050, Y1 X322516MMB4SI

Commit message: Changed all "LCSC" fields to "JLCPCB"
Parts:
- C1, C18, C22, C23, C24, C3, C30, C5, C8, C9: JLCPCB (none) -> C14663; LCSC C14663 -> (none)
- C10, C7: JLCPCB (none) -> C1634; LCSC C1634 -> (none)
- C12, C13, C15, C17: JLCPCB (none) -> C1525; LCSC C1525 -> (none)
- C16, C2, C4, C6: JLCPCB (none) -> C15849; LCSC C15849 -> (none)
- C19, C26: JLCPCB (none) -> C57112; LCSC C57112 -> (none)
- C20, C21: JLCPCB (none) -> C28323; LCSC C28323 -> (none)
- C25: JLCPCB (none) -> C1604; LCSC C1604 -> (none)
- C27, C31, C32: JLCPCB (none) -> C96446; LCSC C96446 -> (none)
- D1: JLCPCB (none) -> C2297; LCSC C2297 -> (none)
- D3: JLCPCB (none) -> C72038; LCSC C72038 -> (none)
- D5, D6: JLCPCB (none) -> C191023; LCSC C191023 -> (none)
- D7, D8: JLCPCB (none) -> C2286; LCSC C2286 -> (none)
- FB1: JLCPCB (none) -> C1015; LCSC C1015 -> (none)
- J4: JLCPCB (none) -> C2936184; LCSC C2936184 -> (none)
- Q1, Q4: JLCPCB (none) -> C20917; LCSC C20917 -> (none)
- Q2, Q5: JLCPCB (none) -> C35349; LCSC C35349 -> (none)
- R1, R3: JLCPCB (none) -> C23162; LCSC C23162 -> (none)
- R10: JLCPCB (none) -> C22984; LCSC C22984 -> (none)
- R11, R19, R2, R25, R4, R6: JLCPCB (none) -> C25804; LCSC C25804 -> (none)
- R12, R13, R17, R21, R22, R23: JLCPCB (none) -> C25803; LCSC C25803 -> (none)
- R18, R20, R24, R26, R27, R9: JLCPCB (none) -> C23193; LCSC C23193 -> (none)
- R28, R29: JLCPCB (none) -> C23186; LCSC C23186 -> (none)
- R30: JLCPCB (none) -> C31850; LCSC C31850 -> (none)
- R31: JLCPCB (none) -> C25819; LCSC C25819 -> (none)
- R32: JLCPCB (none) -> C21190; LCSC C21190 -> (none)
- R5: JLCPCB (none) -> C22978; LCSC C22978 -> (none)
- R7: JLCPCB (none) -> C23228; LCSC C23228 -> (none)
- R8: JLCPCB (none) -> C22843; LCSC C22843 -> (none)
- SW1, SW2: JLCPCB (none) -> C318884; LCSC C318884 -> (none)
- U1: JLCPCB (none) -> C2887190; LCSC C2887190 -> (none)
- U11: JLCPCB (none) -> C6568; LCSC C6568 -> (none)
- U12: JLCPCB (none) -> C6186; LCSC C6186 -> (none)
- U2: Digi-Key_PN 223-1198-1-ND -> (none); Digikey (none) -> 223-1198-1-ND
- U3: JLCPCB (none) -> C97521; LCSC C97521 -> (none)
- U4, U5, U7: JLCPCB (none) -> C2869734; LCSC C2869734 -> (none)
- U6: JLCPCB (none) -> C8304; LCSC C8304 -> (none)
- U8: JLCPCB (none) -> C484409; LCSC C484409 -> (none)
- U9: JLCPCB (none) -> C24112; LCSC C24112 -> (none)
- Y1: JLCPCB (none) -> C13738; LCSC C13738 -> (none)
