File: Schematics/GPS_Module/GPS_Module.kicad_pcb (KiCad board)
At the start: 4 copper layers, 69.5 x 60 mm, 70 parts, among them J1 GT8E-6P-2H(55), J2 SWD_01x04_Pin, J4 Stack Male Edge Connector, J6 USB_C_Female_USB2_Small, SW1 SW_STM_RESET, SW2 SW_STM_BOOT_MODE, U1 STM32F103CBT6, U10 AMS1117-3.3, U2 CP2102N-Axx-xQFN28, U3 W25Q128JVS, U4 LM66100DCKR, U5 LM66100DCKR, U6 LM66100DCKR, U7 TPM8837C-SO1R, U9 ISO1042BQDWVR, Y1 X322516MMB4SI

Commit message: Finalized silkscreen
Other:
- board text added: "GPS Module Rev 2.0 QRET Mar 2025 Tristan Alderson Kennan Bays"
- board text added: "GPS Module V2.0"
- board text added: "NASONOV"
- board text removed: "CHEDDAR V2.0"
- board text removed: "Cheddar Rev 2.0 QRET Mar 2025 Tristan Alderson Kennan Bays"
- board text removed: "GPS Module"
Changed lines of the file:
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@@
       (plot_on_all_layers_selection 0x0000000_00000000)
       (disableapertmacros false)
-      (usegerberextensions false)
-      (usegerberattributes true)
-      (usegerberadvancedattributes true)
-      (creategerberjobfile true)
+      (usegerberextensions true)
+      (usegerberattributes false)
+      (usegerberadvancedattributes false)
+      (creategerberjobfile false)
       (dashed_line_dash_ratio 12.000000)
       (dashed_line_gap_ratio 3.000000)
@@
       (plotinvisibletext false)
       (sketchpadsonfab false)
-      (subtractmaskfromsilk false)
+      (subtractmaskfromsilk true)
       (outputformat 1)
       (mirror false)
-      (drillshape 1)
+      (drillshape 0)
       (scaleselection 1)
-      (outputdirectory "")
+      (outputdirectory "gerbers/")
     )
   )
@@
     (fp_line (start 1 0.625) (end -1 0.625)
       (stroke (width 0.1) (type solid)) (layer "F.Fab"))
-    (pad "1" smd roundrect (at -0.9125 0 180) (size 1.025 1.4) (layers "F.Cu" "F.Paste" "F.Mask") (roundrect_rratio 0.243902)
+    (pad "1" smd roundrect (at -0.9125 0 180) (size 1.025 1.4) (layers "F.Cu" "F.Paste" "F.Mask") (roundrect_rratio 0.243902439)
       (net 13 "+3.3VA") (pintype "passive"))
-    (pad "2" smd roundrect (at 0.9125 0 180) (size 1.025 1.4) (layers "F.Cu" "F.Paste" "F.Mask") (roundrect_rratio 0.243902)
+    (pad "2" smd roundrect (at 0.9125 0 180) (size 1.025 1.4) (layers "F.Cu" "F.Paste" "F.Mask") (roundrect_rratio 0.243902439)
       (net 11 "+3.3V") (pintype "passive"))
     (model "${KICAD6_3DMODEL_DIR}/Resistor_SMD.3dshapes/R_0805_2012Metric.wrl"
@@
     (effects (font (size 1.4 1.4) (thickness 0.25) bold) (justify left bottom mirror))
   )
-  (gr_text "Cheddar Rev 2.0\nQRET Mar 2025\n\nTristan Alderson\n    Kennan Bays" (at 56.9 29.2) (layer "B.SilkS")
+  (gr_text "GPS Module Rev 2.0\nQRET Mar 2025\n\nTristan Alderson\n    Kennan Bays" (at 56.9 29.2) (layer "B.SilkS")
     (effects (font (size 1.5 1.5) (thickness 0.25)) (justify top mirror))
   )
@@
     (effects (font (size 1.4 1.4) (thickness 0.25) bold) (justify left bottom))
   )
-  (gr_text "GPS Module" (at 27.5 76.149999 90) (layer "F.SilkS" knockout)
+  (gr_text "GPS Module V2.0" (at 27.5 76.149999 90) (layer "F.SilkS" knockout)
     (effects (font (size 1.5 1.5) (thickness 0.3) bold) (justify left bottom))
   )
@@
     (effects (font (size 1.2 1.2) (thickness 0.2) bold) (justify bottom))
   )
-  (gr_text "CHEDDAR V2.0" (at 24.95 76.149998 90) (layer "F.SilkS" knockout)
+  (gr_text "NASONOV" (at 24.95 76.149998 90) (layer "F.SilkS" knockout)
     (effects (font (size 1.5 1.5) (thickness 0.3) bold) (justify left bottom))
   )
