File: Schematics/GS_Mainboard/GS_Mainboard.kicad_sch (KiCad schematic)
At the start: 154 parts, among them J1 SWD Header, J10 GPIO, J11 AUX_PWR, J12 SRC_IND, J13 BATT1, J14 BATT2, J15 SWITCH, J16 BUTTS, J17 POWER, J2 RASPI, J3 RGB_OUT, J4 RGB_IN, J5 RGB_OUT, J6 FAN1, J7 FAN2, J8 RGB12V, J9 RTX_PWR, Q1 AO3400A, Q1 AO4447A, Q10 AO3400A, Q11 AO3400A, Q12 AO4406A, Q2 AO3400A, Q3 AO3400A, Q4 AO3400A, Q5 AO3400A, Q7 AO3400A, Q9 AO4406A, SW1 SW_STM_RESET, SW2 SW_STM_BOOT_MODE, U2 LMR51430XDDCR, U3 K7805JT-500R3, U4 296-LMR51450FNDRRRCT-ND, U4 STM32F103C8T6, U5 LM66100DCKR, U6 LM66100DCKR, U7 LM74700QDDFRQ1, U8 LM74700QDDFRQ1, U9 ACS37041KLHBLT-010B3

Commit message: Finalized PCB layout
Parts:
- removed U3: K7805JT-500R3, footprints:K7805JT_500R3, symbol K7805JT_500R3:K7805JT-500R3
- added U3: K78L03-500R3, footprints:K78Lxx-500R3_MNS_SIP3, symbol Regulator_Linear:LM7805_TO220
- C14: Digikey C15127 -> 565-EKYC250ELL202MK20S-ND
- J3: value RGB_OUT -> ARGB_OUT
Connections:
- net GND2 is gone; now on net GND: C14.2, C46.2, U9.3 (GND)
- net +12V: now also J8.4 (Pin_4); no longer J8.1 (Pin_1)
- net +BATT: now also U3.1 (VI)
- net 12V_SENSE: now also U4.15 (PA5); no longer U4.14 (PA4)
- net BUTT_1: now also J16.6 (Pin_6); no longer J16.2 (Pin_2)
- net BUTT_2: now also J16.5 (Pin_5), U4.45 (PB8); no longer J16.3 (Pin_3), U4.43 (PB7)
- net BUTT_3: now also U4.43 (PB7); no longer U4.45 (PB8)
- net GND: now also C30.2, J16.3 (Pin_3), U6.2 (GND), U3.2 (GND); no longer J16.5 (Pin_5)
- net LID_SENSE: now also J16.2 (Pin_2); no longer J16.6 (Pin_6)
- net PSU_TEMP: now also U4.14 (PA4); no longer U4.15 (PA5)
- net RGB12_B: now also R24.1, R25.2, U4.39 (PB3); no longer R22.1, R23.2, U4.41 (PB5)
- net RGB12_G: now also R22.1, R23.2; no longer R20.1, R21.2
- net RGB12_R: now also R20.1, R21.2, U4.41 (PB5); no longer R24.1, R25.2, U4.39 (PB3)
- net SCL: now also J10.5 (Pin_5); no longer J10.6 (Pin_6)
- net SDA: now also J10.6 (Pin_6); no longer J10.5 (Pin_5)
- net SWCLK: now also J1.3 (Pin_3); no longer J1.4 (Pin_4)
- net SWDIO: now also J1.4 (Pin_4); no longer J1.3 (Pin_3)
- net V_BUCK: now also U3.3 (VO)
- net 12V_FB: now reaches R10.2, R11.1, U2.4 (FB)
- net B: now reaches Q4.3 (D)
- net B: now also J8.1 (Pin_1); no longer J8.2 (Pin_2)
- net 5V_FB: now reaches C11.2, R10.2, R11.1, U4.7 (FB)
- net 5V_L_A: now reaches C7.1, L2.1, U4.1 (SW), U4.2 (SW__1), U4.3 (SW__2)
- net B2_EN: now reaches J12.3 (Pin_3), R31.1
- net VRX+: now reaches J9.2 (Pin_2), Q1.5 (D), Q1.6 (D), Q1.7 (D), Q1.8 (D)
- net R: now reaches Q2.3 (D)
- net R: now also J8.3 (Pin_3); no longer J8.4 (Pin_4)
- net AUX+: now reaches J11.2 (Pin_2), Q1.5 (D), Q1.6 (D), Q1.7 (D), Q1.8 (D)
- net G: now reaches Q3.3 (D)
- net G: now also J8.2 (Pin_2); no longer J8.3 (Pin_3)
- net B1_EN: now reaches J12.2 (Pin_2), R30.1
- net GPIO1 renamed PB0
- net PB0: now also J10.3 (Pin_3); no longer J10.4 (Pin_4)
- net GPIO2 renamed PB1
- net PB1: now also J10.4 (Pin_4); no longer J10.3 (Pin_3)
Other:
- title: Ground Station Mainboard -> Ground Station Mainboard (Bondsmith)
- moved on the sheet: J12
