File: Schematics/BackplaneSmall/BackplaneAltimeterTest.kicad_pcb (KiCad board)
At the start: 2 copper layers, 69.5 x 47 mm, 7 parts, among them J1 Edge Connector (SLOT 1), J2 Edge Connector (SLOT 2)

Commit message: UpdatedBackplaneCANBusResistors
Parts:
- added R2: 120R, Resistor_SMD:R_0805_2012Metric_Pad1.20x1.40mm_HandSolder, F.Cu at (29.5, 43.0)
- renumbered H5 to H3, H6 to H4
Routing:
- net CAN_H: track 26.6 -> 48.5 mm
- net CAN_L: track 27.2 -> 48.6 mm
